File: CAD/KiCad/librem5_mainboard/03_CPU_PWR.kicad_sch (KiCad schematic)
At the start: 141 parts, among them U101 MIMX8MQ6DVAJZAA_BGA621

Commit message: Use KiCad's new PADS importer/converter tool to go directly from PADS ascii to KiCad 10, place this newly converted project in CAD/PADS/librem5_mainboard/librem5_mainboard_kicad_conversion/, keep the previous converted project that's in CAD/KiCad/librem5_mainboard/ and update it to also use KiCad 10
The one in CAD/KiCad/ seems to be a bit better but this newly converted
project is available in case it might have some improvements (e.g. in
cross-probing or some other more accurate details). Either one (or both)
may be used to completely move the project over to KiCad.

Signed-off-by: Eric Kuzmenko <eric.kuzmenko@puri.sm>
Parts:
- C1, C102, C147, C148, C149, C150, C151, C152, C178, C179, C180, C182, C184, C185, C186, C187, C188, C189, C19, C190, C191, C192, C193, C194, C195, C196, C197, C198, C199, C2, C221, C3, C339, C6, C8: value C0201 -> 104; DESCRIPTION CAP CER 0.1uF 6V3 20% X5R 0201 -> (none); VALUE 104 -> (none)
- C10, C11, C12, C4, C5, C9, C92: value C0402 -> 4.7UF; DESCRIPTION CAP CER 4.7uF 6V3 20% X5R 0402 -> (none); VALUE 4.7UF -> (none)
- C101, C103, C104, C105, C106, C107, C109, C111, C112, C113, C118, C119, C120, C121, C122, C123, C124, C125, C126, C127, C128, C131, C132, C134, C139, C140, C144, C145, C146, C153, C154, C155, C156, C157, C158, C159, C160, C161, C162, C163, C164, C177, C20, C21, C22, C23, C24, C27, C28, C29, C31, C32, C34, C35, C36: value C0201 -> 105; DESCRIPTION CAP CER 1uF 6V3 20% X5R 0201 -> (none); VALUE 105 -> (none)
- C108, C110, C114, C115, C117, C129, C130, C133, C135, C136, C137, C138, C33: value C0201 -> 103; DESCRIPTION CAP CER 0.01uF 25V 20% X5R 0201 -> (none); VALUE 103 -> (none)
- C116, C13, C14, C15, C16, C165, C166, C167, C168, C169, C17, C170, C171, C172, C173, C174, C175, C176, C18: value C0603 -> 22UF; DESCRIPTION CAP CER 22uF 6V3 20% X5R 0603 -> (none); VALUE 22UF -> (none)
- C181, C183: value C0201 -> NC; DESCRIPTION Z Resistor Chip 0201 0R Ohm 1/16W 1% RALEC -> (none); VALUE NC -> (none)
- L104: value BEAD-0201 -> NC; DESCRIPTION Z FB 240ohm@100MHz DCR0.41ohm 0.35A T:0.3mm -> (none); VALUE NC -> (none)
- L13, L15, L19, L29, L30, L39: value BEAD-0201 -> 10; DESCRIPTION FB 240ohm@100MHz DCR0.41ohm 0.35A T:0.3mm -> (none); VALUE 10 -> (none)
- R61: value RES_2 -> 10; DESCRIPTION Resistor Chip 0201 10R Ohm 1/16W 1% RALEC -> (none); VALUE 10 -> (none)
- R62: value RES_2 -> NC; DESCRIPTION Z Resistor Chip 0201 10K Ohm 1/16W 1% RALEC -> (none); VALUE NC -> (none)
- U101: value MIMX8MQ6DVAJZAA_BGA621 -> MIMX8MQ6DVAJZAB; DESCRIPTION IC MIMX8MQ6DVAJZAB i.MX8M Quad Cortex-A53 Processors 1.5GHz -> (none); VALUE MIMX8MQ6DVAJZAB -> (none)
