File: CAD/KiCad/librem5_mainboard/04_LPDDR4.kicad_sch (KiCad schematic)
At the start: 66 parts, among them U101 MIMX8MQ6DVAJZAA_BGA621, U201 MT53B768M32D4NQ_200P

Commit message: Use KiCad's new PADS importer/converter tool to go directly from PADS ascii to KiCad 10, place this newly converted project in CAD/PADS/librem5_mainboard/librem5_mainboard_kicad_conversion/, keep the previous converted project that's in CAD/KiCad/librem5_mainboard/ and update it to also use KiCad 10
The one in CAD/KiCad/ seems to be a bit better but this newly converted
project is available in case it might have some improvements (e.g. in
cross-probing or some other more accurate details). Either one (or both)
may be used to completely move the project over to KiCad.

Signed-off-by: Eric Kuzmenko <eric.kuzmenko@puri.sm>
Parts:
- C201, C206, C211: value C0603 -> 22UF; DESCRIPTION CAP CER 22uF 6V3 20% X5R 0603 -> (none); VALUE 22UF -> (none)
- C202, C203, C204, C205, C207, C208, C209, C210, C212, C213, C214, C215, C217: value C0402 -> 4.7UF; DESCRIPTION CAP CER 4.7uF 6V3 20% X5R 0402 -> (none); VALUE 4.7UF -> (none)
- C216: value C0201 -> 104; DESCRIPTION CAP CER 0.1uF 6V3 20% X5R 0201 -> (none); VALUE 104 -> (none)
- C218, C219, C351, C352, C356, C388, C396, C397, C398, C399, C400, C406, C407, C408, C409, C410, C411, C412, C413, C414, C415, C416, C417, C418, C419, C420, C421, C422, C423, C424, C427, C428, C429, C430, C431, C432, C433: value C0201 -> 105; DESCRIPTION CAP CER 1uF 6V3 20% X5R 0201 -> (none); VALUE 105 -> (none)
- R201, R202: value RES_2 -> 150; DESCRIPTION Resistor Chip 0201 150R Ohm 1/16W 1% RALEC -> (none); VALUE 150 -> (none)
- R203, R204, R205: value RES_2 -> 240; DESCRIPTION Resistor Chip 0201 240R Ohm 1/16W 1% RALEC -> (none); VALUE 240 -> (none)
- R206, R207, R208: value RES_2 -> 10K; DESCRIPTION Resistor Chip 0201 10K Ohm 1/16W 1% RALEC -> (none); VALUE 10K -> (none)
- R209, R210: value RES_2 -> 1.5K; DESCRIPTION Resistor Chip 0201 1.5K Ohm 1/16W 1% RALEC -> (none); VALUE 1.5K -> (none)
- U101: value MIMX8MQ6DVAJZAA_BGA621 -> MIMX8MQ6DVAJZAB; DESCRIPTION IC MIMX8MQ6DVAJZAB i.MX8M Quad Cortex-A53 Processors 1.5GHz -> (none); VALUE MIMX8MQ6DVAJZAB -> (none)
- U201: value MT53B768M32D4NQ_200P -> MT53E768M32D4DT-053 WT:E; DESCRIPTION IC MEM MOBILE LPDDR4 SDRAM 768 Meg x 32 4CH X16 I/O 1.1V AU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 -> (none); VALUE MT53E768M32D4DT-053 WT:E -> (none)
