File: CAD/KiCad/librem5_mainboard/05_CPU_IO.kicad_sch (KiCad schematic)
At the start: 26 parts, among them Q4 2SK3018, Q5 2SK3018, Q8 2SK3018, U101 MIMX8MQ6DVAJZAA_BGA621, U3 NTBA104_XQFN12

Commit message: Use KiCad's new PADS importer/converter tool to go directly from PADS ascii to KiCad 10, place this newly converted project in CAD/PADS/librem5_mainboard/librem5_mainboard_kicad_conversion/, keep the previous converted project that's in CAD/KiCad/librem5_mainboard/ and update it to also use KiCad 10
The one in CAD/KiCad/ seems to be a bit better but this newly converted
project is available in case it might have some improvements (e.g. in
cross-probing or some other more accurate details). Either one (or both)
may be used to completely move the project over to KiCad.

Signed-off-by: Eric Kuzmenko <eric.kuzmenko@puri.sm>
Parts:
- C46: value C0402 -> 4.7UF; DESCRIPTION CAP CER 4.7uF 6V3 20% X5R 0402 -> (none); VALUE 4.7UF -> (none)
- C68: value C0402 -> 225; DESCRIPTION CAP CER 2.2uF 35V 20% X5R 0402 -> (none); VALUE 225 -> (none)
- D16, D20: value DIODE_SCHTKY_0 -> RB751G-40; DESCRIPTION Diode schottky SOD723 40V 30mA mark:5 RB751G-40 ³¤µç -> (none); VALUE RB751G-40 -> (none)
- Q4, Q5, Q8: value 2SK3018 -> RYU002N05; DESCRIPTION TRAN NMOS SW 0.9V DRIVE 50V UMT3 -> (none); VALUE RYU002N05 -> (none)
- R104, R219, R221, R225, R226: value RES_2 -> 10; DESCRIPTION Resistor Chip 0201 10R Ohm 1/16W 1% RALEC -> (none); VALUE 10 -> (none)
- R2, R3: value RES_2 -> 4.7K; DESCRIPTION Resistor Chip 0201 4.7K Ohm 1/16W 1% RALEC -> (none); VALUE 4.7K -> (none)
- R27: value RES_2 -> NC; DESCRIPTION Z Resistor Chip 0201 10K Ohm 1/16W 1% RALEC -> (none); VALUE NC -> (none)
- R301, R302, R303, R304, R305, R306, R307, R308: value RES_2 -> 2.2K; DESCRIPTION Resistor Chip 0201 2.2K Ohm 1/16W 1% RALEC -> (none); VALUE 2.2K -> (none)
- R31: value RES_2 -> 47K; DESCRIPTION Resistor Chip 0201 47K Ohm 1/16W 1% RALEC -> (none); VALUE 47K -> (none)
- U101: value MIMX8MQ6DVAJZAA_BGA621 -> MIMX8MQ6DVAJZAB; DESCRIPTION IC MIMX8MQ6DVAJZAB i.MX8M Quad Cortex-A53 Processors 1.5GHz -> (none); VALUE MIMX8MQ6DVAJZAB -> (none)
- U3: value NTBA104_XQFN12 -> NC; DESCRIPTION Z IC Dual Supply Buffer 4BIT NTB0104GU12 -> (none); VALUE NC -> (none)
