File: CAD/KiCad/librem5_mainboard/06_CPU_MISC_RTC.kicad_sch (KiCad schematic)
At the start: 20 parts, among them U101 MIMX8MQ6DVAJZAA_BGA621, U39 RV-4162-C7, Y401 XTAL_13Y, Y402 XTAL_13Y

Commit message: Use KiCad's new PADS importer/converter tool to go directly from PADS ascii to KiCad 10, place this newly converted project in CAD/PADS/librem5_mainboard/librem5_mainboard_kicad_conversion/, keep the previous converted project that's in CAD/KiCad/librem5_mainboard/ and update it to also use KiCad 10
The one in CAD/KiCad/ seems to be a bit better but this newly converted
project is available in case it might have some improvements (e.g. in
cross-probing or some other more accurate details). Either one (or both)
may be used to completely move the project over to KiCad.

Signed-off-by: Eric Kuzmenko <eric.kuzmenko@puri.sm>
Parts:
- C401: value C0201 -> 105; DESCRIPTION CAP CER 1uF 6V3 20% X5R 0201 -> (none); VALUE 105 -> (none)
- C402, C403, C404, C405: value C0201 -> 18PF; DESCRIPTION CAP CER 18PF 25V 20% NPO 0201 -> (none); VALUE 18PF -> (none)
- C4051: value C0201 -> 104; DESCRIPTION CAP CER 0.1uF 6V3 20% X5R 0201 -> (none); VALUE 104 -> (none)
- C448, C450: value C0603 -> 22UF; DESCRIPTION CAP CER 22uF 6V3 20% X5R 0603 -> (none); VALUE 22UF -> (none)
- D22, D8: value DIODE_SCHTKY_0 -> RB751G-40; DESCRIPTION Diode schottky SOD723 40V 30mA mark:5 RB751G-40 ³¤µç -> (none); VALUE RB751G-40 -> (none)
- R127: value RES_2 -> 10; DESCRIPTION Resistor Chip 0201 10R Ohm 1/16W 1% RALEC -> (none); VALUE 10 -> (none)
- R236: value RES_2 -> 100; DESCRIPTION Resistor Chip 0201 100R Ohm 1/16W 1% RALEC -> (none); VALUE 100 -> (none)
- R409: value RES_2 -> 4.7K; DESCRIPTION Resistor Chip 0201 4.7K Ohm 1/16W 1% RALEC -> (none); VALUE 4.7K -> (none)
- R410, R416: value RES_2 -> 10K; DESCRIPTION Resistor Chip 0201 10K Ohm 1/16W 1% RALEC -> (none); VALUE 10K -> (none)
- R419: value RES_2 -> 100K; DESCRIPTION Resistor Chip 0201 100K Ohm 1/16W 1% RALEC -> (none); VALUE 100K -> (none)
- U101: value MIMX8MQ6DVAJZAA_BGA621 -> MIMX8MQ6DVAJZAB; DESCRIPTION IC MIMX8MQ6DVAJZAB i.MX8M Quad Cortex-A53 Processors 1.5GHz -> (none); VALUE MIMX8MQ6DVAJZAB -> (none)
- U39: DESCRIPTION IC Real Time Clock Moudule with I2C Bus -> (none); VALUE RV-4162-C7 -> (none)
- Y401: value XTAL_13Y -> 25MHz; DESCRIPTION CLOCK Crystal 25MHz 9pF +-30PPM/ -> (none); VALUE 25MHz -> (none)
- Y402: value XTAL_13Y -> 27MHz; DESCRIPTION CLOCK Crystal 27MHz 9pF +-30PPM/ -> (none); VALUE 27MHz -> (none)
