File: CAD/KiCad/librem5_mainboard/07_CPU_PHY.kicad_sch (KiCad schematic)
At the start: 18 parts, among them U101 MIMX8MQ6DVAJZAA_BGA621, Y501 NX5427001Z_6P

Commit message: Use KiCad's new PADS importer/converter tool to go directly from PADS ascii to KiCad 10, place this newly converted project in CAD/PADS/librem5_mainboard/librem5_mainboard_kicad_conversion/, keep the previous converted project that's in CAD/KiCad/librem5_mainboard/ and update it to also use KiCad 10
The one in CAD/KiCad/ seems to be a bit better but this newly converted
project is available in case it might have some improvements (e.g. in
cross-probing or some other more accurate details). Either one (or both)
may be used to completely move the project over to KiCad.

Signed-off-by: Eric Kuzmenko <eric.kuzmenko@puri.sm>
Parts:
- C501: value C0201 -> 104; DESCRIPTION CAP CER 0.1uF 6V3 20% X5R 0201 -> (none); VALUE 104 -> (none)
- R189, R508, R509: value RES_2 -> 100K; DESCRIPTION Resistor Chip 0201 100K Ohm 1/16W 1% RALEC -> (none); VALUE 100K -> (none)
- R190, R199: value RES_2 -> 2.2K; DESCRIPTION Resistor Chip 0201 2.2K Ohm 1/16W 1% RALEC -> (none); VALUE 2.2K -> (none)
- R200: value RES_2 -> 27K; DESCRIPTION Resistor Chip 0201 27K Ohm 1/16W 1% RALEC -> (none); VALUE 27K -> (none)
- R503: value RES_2 -> 499; DESCRIPTION Resistor Chip 0201 499 Ohm 1/16W 1% RALEC -> (none); VALUE 499 -> (none)
- R504, R506: value RES_2 -> 200; DESCRIPTION Resistor Chip 0201 200R Ohm 1/16W 1% RALEC -> (none); VALUE 200 -> (none)
- R505: value RES_2 -> 15K; DESCRIPTION Resistor Chip 0201 15K Ohm 1/16W 1% RALEC -> (none); VALUE 15K -> (none)
- R507: value RES_2 -> 10K; DESCRIPTION Resistor Chip 0201 10K Ohm 1/16W 1% RALEC -> (none); VALUE 10K -> (none)
- R510, R511: value RES_2 -> 0; DESCRIPTION Resistor Chip 0201 0R Ohm 1/16W 1% RALEC -> (none); VALUE 0 -> (none)
- R98: value RES_2 -> 1K; DESCRIPTION Resistor Chip 0201 1K Ohm 1/16W 1% RALEC -> (none); VALUE 1K -> (none)
- TC8: value TEST-POINT -> M3; DESCRIPTION Z -> (none); VALUE M3 -> (none)
- U101: value MIMX8MQ6DVAJZAA_BGA621 -> MIMX8MQ6DVAJZAB; DESCRIPTION IC MIMX8MQ6DVAJZAB i.MX8M Quad Cortex-A53 Processors 1.5GHz -> (none); VALUE MIMX8MQ6DVAJZAB -> (none)
- Y501: value NX5427001Z_6P -> NX5427001Z; DESCRIPTION OSC 27MHz HCSL 3.3V 5X3.2MM SMT -> (none); VALUE NX5427001Z -> (none)
