File: CAD/KiCad/librem5_mainboard/08_EMMC.kicad_sch (KiCad schematic)
At the start: 16 parts, among them U601 MTFC8GACAEAM_VFBGA_0

Commit message: Use KiCad's new PADS importer/converter tool to go directly from PADS ascii to KiCad 10, place this newly converted project in CAD/PADS/librem5_mainboard/librem5_mainboard_kicad_conversion/, keep the previous converted project that's in CAD/KiCad/librem5_mainboard/ and update it to also use KiCad 10
The one in CAD/KiCad/ seems to be a bit better but this newly converted
project is available in case it might have some improvements (e.g. in
cross-probing or some other more accurate details). Either one (or both)
may be used to completely move the project over to KiCad.

Signed-off-by: Eric Kuzmenko <eric.kuzmenko@puri.sm>
Parts:
- C601, C605: value C0402 -> 4.7UF; DESCRIPTION CAP CER 4.7uF 6V3 20% X5R 0402 -> (none); VALUE 4.7UF -> (none)
- C602, C603, C604, C606, C607, C610: value C0201 -> 104; DESCRIPTION CAP CER 0.1uF 6V3 20% X5R 0201 -> (none); VALUE 104 -> (none)
- C611: value C0201 -> 105; DESCRIPTION CAP CER 1uF 6V3 20% X5R 0201 -> (none); VALUE 105 -> (none)
- R601, R602, R603: value RES_2 -> 4.7K; DESCRIPTION Resistor Chip 0201 4.7K Ohm 1/16W 1% RALEC -> (none); VALUE 4.7K -> (none)
- R616, R617, R621: value RES_2 -> 0; DESCRIPTION Resistor Chip 0201 0R Ohm 1/16W 1% RALEC -> (none); VALUE 0 -> (none)
- U601: value MTFC8GACAEAM_VFBGA_0 -> THGBMHG8C2LBAIR; DESCRIPTION IC MEM NAND FLASH 32GB MMC 5.1 THGBMHG8C2LBAIR FBGA153 -> (none); VALUE THGBMHG8C2LBAIR -> (none)
