File: CAD/KiCad/librem5_mainboard/09_PMIC.kicad_sch (KiCad schematic)
At the start: 112 parts, among them U1 BD71837-24, U704 UM805_4P, Y1 32768-2

Commit message: Use KiCad's new PADS importer/converter tool to go directly from PADS ascii to KiCad 10, place this newly converted project in CAD/PADS/librem5_mainboard/librem5_mainboard_kicad_conversion/, keep the previous converted project that's in CAD/KiCad/librem5_mainboard/ and update it to also use KiCad 10
The one in CAD/KiCad/ seems to be a bit better but this newly converted
project is available in case it might have some improvements (e.g. in
cross-probing or some other more accurate details). Either one (or both)
may be used to completely move the project over to KiCad.

Signed-off-by: Eric Kuzmenko <eric.kuzmenko@puri.sm>
Parts:
- C244, C278: value C0201 -> 10P; DESCRIPTION CAP CER 10PF 6V3 20% NPO 0201 -> (none); VALUE 10P -> (none)
- C279, C280, C322, C383, C732, C738, C744, C752, C761: value C0603 -> NC; DESCRIPTION Z CAP CER 22uF 6V3 20% X5R 0603 -> (none); VALUE NC -> (none)
- C282, C311, C312, C480, C542, C729, C737, C743, C747, C749, C750, C751, C754, C755, C757, C759: value C0402 -> 4.7UF; DESCRIPTION CAP CER 4.7uF 6V3 20% X5R 0402 -> (none); VALUE 4.7UF -> (none)
- C284, C285, C313, C521, C710, C722, C723, C725, C731, C739, C741, C742, C745, C753, C760, C769, C77, C775: value C0603 -> 22UF; DESCRIPTION CAP CER 22uF 6V3 20% X5R 0603 -> (none); VALUE 22UF -> (none)
- C381, C384, C385, C387, C389, C445, C446, C522, C523, C717, C728, C746: value C0201 -> 105; DESCRIPTION CAP CER 1uF 6V3 20% X5R 0201 -> (none); VALUE 105 -> (none)
- C447: value C0201 -> 103; DESCRIPTION CAP CER 0.01uF 25V 20% X5R 0201 -> (none); VALUE 103 -> (none)
- C736: value C0603 -> 22UF; DESCRIPTION CAP CER 4.7UF 6.3V 10% X5R 0603 -> (none); VALUE 22UF -> (none)
- C740: value C0603 -> 10uF; DESCRIPTION CAP CER 4.7UF 6.3V 10% X5R 0603 -> (none); VALUE 10uF -> (none)
- C758: value C0201 -> 104; DESCRIPTION CAP CER 0.1uF 6V3 20% X5R 0201 -> (none); VALUE 104 -> (none)
- D21, D3: value DIODE_SCHTKY_0 -> RB751G-40; DESCRIPTION Diode schottky SOD723 40V 30mA mark:5 RB751G-40 ³¤µç -> (none); VALUE RB751G-40 -> (none)
- L32: value INDUCTOR -> WPN252012H1R0MT; DESCRIPTION IND PWR 1uH@1MHZ 4.2A 20% SMT -> (none); VALUE WPN252012H1R0MT -> (none)
- L702, L703, L704, L705, L706, L707, L710: value INDUCTOR -> WPN252012ER47MT; DESCRIPTION IND PWR 0.47uH@1MHZ 4.7A 20% SMT -> (none); VALUE WPN252012ER47MT -> (none)
- R1, R90, R94: value RES_2 -> 0; DESCRIPTION Resistor Chip 0201 0R Ohm 1/16W 1% RALEC -> (none); VALUE 0 -> (none)
- R140, R152, R167, R168: value CURRENT_R -> 20m OHM; DESCRIPTION Resistor Chip 0603 20m Ohm 1/10W 1% RALEC -> (none); VALUE 20m OHM -> (none)
- R15, R157, R4, R92: value RES_2 -> 10K; DESCRIPTION Resistor Chip 0201 10K Ohm 1/16W 1% RALEC -> (none); VALUE 10K -> (none)
- R185: value RES_2 -> 100; DESCRIPTION Resistor Chip 0201 100R Ohm 1/16W 1% RALEC -> (none); VALUE 100 -> (none)
- R186: value RES_2 -> 560K; DESCRIPTION Resistor Chip 0201 560K Ohm 1/16W 1% RALEC -> (none); VALUE 560K -> (none)
- R259, R260: value R_0201 -> 0R; VALUE 0R -> (none)
- R91: value RES_2 -> NC; DESCRIPTION Z Resistor Chip 0201 10K Ohm 1/16W 1% RALEC -> (none); VALUE NC -> (none)
- R93: value RES_2 -> 47K; DESCRIPTION Resistor Chip 0201 47K Ohm 1/16W 1% RALEC -> (none); VALUE 47K -> (none)
- TC13, TC15, TC4, TC62, TC71, TC72, TC81, TC82, TV21, TV22, TV23, TV60, TV61, TV62, TV63, TV64, TV65, TV66, TV67, TV68, TV69: value TEST-POINT -> M3; DESCRIPTION Z -> (none); VALUE M3 -> (none)
- U1: value BD71837-24 -> BD71837MWV; DESCRIPTION IC POWER MANAGEMENT BUCK 8CH LDO 7CH -0.3-5.5V -> (none); VALUE BD71837MWV -> (none)
- U704: value UM805_4P -> UM805RE; DESCRIPTION IC VOLT MONITOR 2.63V VTH RST 1-5.5V SOT143 -> (none); VALUE UM805RE -> (none)
- Y1: value 32768-2 -> 32768 10pF +-20PPM; DESCRIPTION CLOCK Crystal 1.5~3.6V ASH7K-32.768KHz-T?? -> (none); VALUE 32768 10pF +-20PPM -> (none)
