File: CAD/KiCad/librem5_mainboard/10_BOOT_CFG.kicad_sch (KiCad schematic)
At the start: 82 parts, among them J1 CON-6PIN-OK-501F006-13, Q10 2SK3018, Q11 2SK3018, Q14 2SK3018, Q18 2SK3018, Q19 AP2302, Q7 2SK3018, SW3 HOLD-3P, SW5 HOLD-3P, SW7 HOLD-3P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

Commit message: Use KiCad's new PADS importer/converter tool to go directly from PADS ascii to KiCad 10, place this newly converted project in CAD/PADS/librem5_mainboard/librem5_mainboard_kicad_conversion/, keep the previous converted project that's in CAD/KiCad/librem5_mainboard/ and update it to also use KiCad 10
The one in CAD/KiCad/ seems to be a bit better but this newly converted
project is available in case it might have some improvements (e.g. in
cross-probing or some other more accurate details). Either one (or both)
may be used to completely move the project over to KiCad.

Signed-off-by: Eric Kuzmenko <eric.kuzmenko@puri.sm>
Parts:
- D1, D4: value ZLLS400 -> B5817WS; DESCRIPTION DIODE Schottky Barrier Diode SOD323 -> (none); VALUE B5817WS -> (none)
- D11, D13, D15, D18, D23, D24, D28, D29, D9: value DIODE_SCHTKY_0 -> RB751G-40; DESCRIPTION Diode schottky SOD723 40V 30mA mark:5 RB751G-40 ³¤µç -> (none); VALUE RB751G-40 -> (none)
- D27: value LED_LRTB_R98G -> LRTB R98G; DESCRIPTION LED Multi CHIPLED -> (none); VALUE LRTB R98G -> (none)
- Q10, Q11, Q14, Q18, Q7: value 2SK3018 -> RYU002N05; DESCRIPTION TRAN NMOS SW 0.9V DRIVE 50V UMT3 -> (none); VALUE RYU002N05 -> (none)
- Q19: DESCRIPTION TRANS MOSFET N-CH 16V 3.6A SOT-23 -> (none); VALUE AP2302 -> (none)
- R118, R126: value RES_2 -> 18R; DESCRIPTION Resistor Chip 0201 1K Ohm 1/16W 1% RALEC -> (none); VALUE 18R -> (none)
- R132: value RES_2 -> 100R; DESCRIPTION Resistor Chip 0201 1K Ohm 1/16W 1% RALEC -> (none); VALUE 100R -> (none)
- R145, R192, R193, R194, R232, R48, R56, R66, R67, R68, R825, R827, R828, R829, R832, R833, R834, R835, R836, R839, R840: value RES_2 -> 47K; DESCRIPTION Resistor Chip 0201 47K Ohm 1/16W 1% RALEC -> (none); VALUE 47K -> (none)
- R156, R191, R213, R624: value RES_2 -> 1K; DESCRIPTION Resistor Chip 0201 1K Ohm 1/16W 1% RALEC -> (none); VALUE 1K -> (none)
- R215: value RES_2 -> 470K; DESCRIPTION Resistor Chip 0201 470K Ohm 1/16W 1% RALEC -> (none); VALUE 470K -> (none)
- R239, R625, R626, R627: value RES_2 -> 100; DESCRIPTION Resistor Chip 0201 100R Ohm 1/16W 1% RALEC -> (none); VALUE 100 -> (none)
- R240: value RES_2 -> 0; DESCRIPTION Resistor Chip 0201 0R Ohm 1/16W 1% RALEC -> (none); VALUE 0 -> (none)
- R241, R803, R811, R815: value RES_2 -> 10K; DESCRIPTION Resistor Chip 0201 10K Ohm 1/16W 1% RALEC -> (none); VALUE 10K -> (none)
- R809, R810, R812, R814, R816, R830, R838: value RES_2 -> NC; DESCRIPTION Z Resistor Chip 0201 10K Ohm 1/16W 1% RALEC -> (none); VALUE NC -> (none)
- R831, R837: value RES_2 -> 100K; DESCRIPTION Resistor Chip 0201 100K Ohm 1/16W 1% RALEC -> (none); VALUE 100K -> (none)
- SW3, SW5, SW7: value HOLD-3P -> EL-MSK02; DESCRIPTION SW SLIDE 7PIN -> (none); VALUE EL-MSK02 -> (none)
- TP13, TP14, TP15: value T_POINT_R -> GND; DESCRIPTION Z -> (none); VALUE GND -> (none)
- TP7: value T_POINT_R -> PWR KEY; DESCRIPTION Z -> (none); VALUE PWR KEY -> (none)
- TP8: value T_POINT_R -> VOL+; DESCRIPTION Z -> (none); VALUE VOL+ -> (none)
- TP9: value T_POINT_R -> VOL-; DESCRIPTION Z -> (none); VALUE VOL- -> (none)
- TVS12, TVS13, TVS14, TVS15, TVS16: value TVS_0402_882 -> PESD3V3S1UL; DESCRIPTION IC ESD 3V3 200pF 30KV SOD882 µ¥Ïò -> (none); VALUE PESD3V3S1UL -> (none)
- TVS29: value TVS_0402_882 -> PESD5V0S1BL; DESCRIPTION IC ESD 5V0 45pF 30KV SOD882 Ë«Ïò -> (none); VALUE PESD5V0S1BL -> (none)
- U47: value SMD-MOTO -> CQ3610BL-100; DESCRIPTION MOTO 2.7V 14000rpm 75mA 33ohm -> (none); VALUE CQ3610BL-100 -> (none)
