File: CAD/KiCad/librem5_mainboard/12_CHARGE_BAT_LED.kicad_sch (KiCad schematic)
At the start: 55 parts, among them J20 CON-3PIN, U14 BQ25895-25, U15 MAX17047_0

Commit message: Use KiCad's new PADS importer/converter tool to go directly from PADS ascii to KiCad 10, place this newly converted project in CAD/PADS/librem5_mainboard/librem5_mainboard_kicad_conversion/, keep the previous converted project that's in CAD/KiCad/librem5_mainboard/ and update it to also use KiCad 10
The one in CAD/KiCad/ seems to be a bit better but this newly converted
project is available in case it might have some improvements (e.g. in
cross-probing or some other more accurate details). Either one (or both)
may be used to completely move the project over to KiCad.

Signed-off-by: Eric Kuzmenko <eric.kuzmenko@puri.sm>
Parts:
- C288, C289, C56: value C0603 -> 22UF; DESCRIPTION CAP CER 22uF 6V3 20% X5R 0603 -> (none); VALUE 22UF -> (none)
- C317, C318, C541, C57: value C0201 -> 105; DESCRIPTION CAP CER 1uF 6V3 20% X5R 0201 -> (none); VALUE 105 -> (none)
- C319, C363, C364, C49: value C0603 -> 10UF; DESCRIPTION CAP CER 10uF 35V 20% X5R 0603 -> (none); VALUE 10UF -> (none)
- C320, C321, C365, C535: value C0402 -> 224; DESCRIPTION CAP CER 0.22uF 35V 20% X5R 0402 -> (none); VALUE 224 -> (none)
- C366, C51: value C0201 -> 104; DESCRIPTION CAP CER 0.1uF 6V3 20% X5R 0201 -> (none); VALUE 104 -> (none)
- C50: value C0201 -> NC; DESCRIPTION Z CAP CER 1uF 6V3 20% X5R 0201 -> (none); VALUE NC -> (none)
- D5: value ZLLS400 -> B5817WS; DESCRIPTION DIODE Schottky Barrier Diode SOD323 -> (none); VALUE B5817WS -> (none)
- L46: value INDUCTOR_IRON_1 -> AMPI0618ED2R2MT; DESCRIPTION IND PWR 2.2UH@100KHZ Isat 8A 20% SMT -> (none); VALUE AMPI0618ED2R2MT -> (none)
- L58, L59: value BEAD-4030 -> PZ3216D600-4R0TF; DESCRIPTION FB 60ohm@100MHz DCR20mohm 4A T:0.85mm -> (none); VALUE PZ3216D600-4R0TF -> (none)
- L60: value BEAD-0402 -> MZAH1005F352-R27TF; DESCRIPTION FB 3500ohm@100MHz 1600ohm@1GHz DCR1ohm 270mA T:0.5mm -> (none); VALUE MZAH1005F352-R27TF -> (none)
- R112, R30, R34, R57: value RES_2 -> 0; DESCRIPTION Resistor Chip 0201 0R Ohm 1/16W 1% RALEC -> (none); VALUE 0 -> (none)
- R113, R114, R196, R20, R22: value RES_2 -> 10K; DESCRIPTION Resistor Chip 0201 10K Ohm 1/16W 1% RALEC -> (none); VALUE 10K -> (none)
- R115: value RES_2 -> 200; DESCRIPTION Resistor Chip 0201 200R Ohm 1/16W 1% RALEC -> (none); VALUE 200 -> (none)
- R116: value RES_2 -> 30.1K; DESCRIPTION Resistor Chip 0201 30.1K Ohm 1/16W 1% RALEC -> (none); VALUE 30.1K -> (none)
- R117: value RES_2 -> 5.23K; DESCRIPTION Resistor Chip 0201 5.23K Ohm 1/16W 1% RALEC -> (none); VALUE 5.23K -> (none)
- R134, R182, R183, R195: value CURRENT_R -> 20m OHM; DESCRIPTION Resistor Chip 0603 20m Ohm 1/10W 1% RALEC -> (none); VALUE 20m OHM -> (none)
- R180, R184, R312: value CURRENT_R -> 5m OHM; DESCRIPTION Resistor Chip 0603 5m Ohm 1/10W 1% RALEC -> (none); VALUE 5m OHM -> (none)
- R21, R29: value RES_2 -> NC; DESCRIPTION Z Resistor Chip 0201 10K Ohm 1/16W 1% RALEC -> (none); VALUE NC -> (none)
- R99: value RES_2 -> 1K; DESCRIPTION Resistor Chip 0201 1K Ohm 1/16W 1% RALEC -> (none); VALUE 1K -> (none)
- TP18, TP20, TP21: value T_POINT_R -> GND; DESCRIPTION Z -> (none); VALUE GND -> (none)
- TV2, TV3, TV4, TV5: value TEST-POINT -> M3; DESCRIPTION Z -> (none); VALUE M3 -> (none)
- U14: value BQ25895-25 -> BQ25895; DESCRIPTION IC i2c Controlled Single Cell 5A Fast Charger for High Inpu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 -> (none); VALUE BQ25895 -> (none)
- U15: value MAX17047_0 -> MAX17055; DESCRIPTION IC 7uA 1cell Fuel Gauge with ModelGauge m5 EZ -> (none); VALUE MAX17055 -> (none)
Connections:
- net N47770321: no longer names the net of R21.1, U15.C2 (THRM)
- net N47847848: no longer names the net of C320.1, U14.21 (BTST)
Other:
- moved on the sheet: C51
