File: CAD/KiCad/librem5_mainboard/13_SENSOR_SMARTCARD.kicad_sch (KiCad schematic)
At the start: 75 parts, among them J9 MICRO-SIMCARD, U16 LSM9DS1, U23 AP2281, U26 VCNL4040, U300 AH3663, U329 STM32L432KC, U330 TXS4555, U4 AP2281, U56 74LVC1G125-SC70-5, U68 NTSX2102GU8_1.4X1.2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

Commit message: Use KiCad's new PADS importer/converter tool to go directly from PADS ascii to KiCad 10, place this newly converted project in CAD/PADS/librem5_mainboard/librem5_mainboard_kicad_conversion/, keep the previous converted project that's in CAD/KiCad/librem5_mainboard/ and update it to also use KiCad 10
The one in CAD/KiCad/ seems to be a bit better but this newly converted
project is available in case it might have some improvements (e.g. in
cross-probing or some other more accurate details). Either one (or both)
may be used to completely move the project over to KiCad.

Signed-off-by: Eric Kuzmenko <eric.kuzmenko@puri.sm>
Parts:
- C143, C223, C224, C331, C354, C425, C426, C438, C79, C80: value C0201 -> 105; DESCRIPTION CAP CER 1uF 6V3 20% X5R 0201 -> (none); VALUE 105 -> (none)
- C254, C334, C357, C358, C359, C48, C512, C81, C82: value C0201 -> 104; DESCRIPTION CAP CER 0.1uF 6V3 20% X5R 0201 -> (none); VALUE 104 -> (none)
- C332, C333: value C0201 -> 6.8PF; DESCRIPTION CAP CER 6.8PF 25V 10% NPO 0201 -> (none); VALUE 6.8PF -> (none)
- C360, C513, C78: value C0402 -> 4.7UF; DESCRIPTION CAP CER 4.7uF 6V3 20% X5R 0402 -> (none); VALUE 4.7UF -> (none)
- C52: value C0201 -> 103; DESCRIPTION CAP CER 0.01uF 25V 20% X5R 0201 -> (none); VALUE 103 -> (none)
- C83: value C0603 -> 22UF; DESCRIPTION CAP CER 22uF 6V3 20% X5R 0603 -> (none); VALUE 22UF -> (none)
- D12, D14, D17: value DIODE_SCHTKY_0 -> RB751G-40; DESCRIPTION Diode schottky SOD723 40V 30mA mark:5 RB751G-40 ³¤µç -> (none); VALUE RB751G-40 -> (none)
- J9: DESCRIPTION Micro sim card p/n:SA0701127150-105 -> (none)
- L22, L56, L64: value BEAD-0402 -> 10 / HPZ1005U121-1R1TF; DESCRIPTION Resistor Chip 0402 10 Ohm 1/16W 1% RALEC -> (none); VALUE 10 / HPZ1005U121-1R1TF -> (none)
- L23: value BEAD-0402 -> HPZ1005U121-1R1TF; DESCRIPTION FB 120ohm@100MHz 100ohm@1GHz DCR0.13ohm 1.1A T:0.5mm -> (none); VALUE HPZ1005U121-1R1TF -> (none)
- L72: value BEAD-0402 -> 0.2 / HPZ1005U121-1R1TF; DESCRIPTION Resistor Chip 0402 0.2 Ohm 1/16W 1% RALEC -> (none); VALUE 0.2 / HPZ1005U121-1R1TF -> (none)
- R105, R108, R141, R165, R19, R217, R220, R224, R229, R233, R52: value RES_2 -> 10K; DESCRIPTION Resistor Chip 0201 10K Ohm 1/16W 1% RALEC -> (none); VALUE 10K -> (none)
- R130, R135, R222: value RES_2 -> NC; DESCRIPTION Z Resistor Chip 0201 10K Ohm 1/16W 1% RALEC -> (none); VALUE NC -> (none)
- R139, R161, R162: value RES_2 -> 0; DESCRIPTION Resistor Chip 0201 0R Ohm 1/16W 1% RALEC -> (none); VALUE 0 -> (none)
- R177, R216, R230, R231, R6: value RES_2 -> 10; DESCRIPTION Resistor Chip 0201 10R Ohm 1/16W 1% RALEC -> (none); VALUE 10 -> (none)
- R179, R214: value RES_2 -> 47K; DESCRIPTION Resistor Chip 0201 47K Ohm 1/16W 1% RALEC -> (none); VALUE 47K -> (none)
- TC1, TC2, TV36, TV37, TV38: value TEST-POINT -> M3; DESCRIPTION Z -> (none); VALUE M3 -> (none)
- TVS8: value TVS_0402_882 -> PESD3V3S1UL; DESCRIPTION IC ESD 3V3 200pF 30KV SOD882 µ¥Ïò -> (none); VALUE PESD3V3S1UL -> (none)
- U16: DESCRIPTION IC 9-axis sensor[LSM9DS1] -> (none); VALUE LSM9DS1 -> (none)
- U23, U4: value AP2281 -> AP2281-3FMG; DESCRIPTION IC SWITCH 80mohm 1.5-6V -> (none); VALUE AP2281-3FMG -> (none)
- U26: value VCNL4040 -> VCNL4040M3OE-H5; DESCRIPTION IC Light Sensor PS and ALS -> (none); VALUE VCNL4040M3OE-H5 -> (none)
- U300: DESCRIPTION IC Hall sensor -> (none); VALUE AH3663 -> (none)
- U329: DESCRIPTION IC Arm Cotex M4 MCU+FPU,100DMIPS, 256KB FLASH,64KB SRAM, US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 -> (none); VALUE STM32L432KC -> (none)
- U330: DESCRIPTION IC SIM¿¨µçÆ½×ª»» -> (none); VALUE TXS4555 -> (none)
- U56: value 74LVC1G125-SC70-5 -> 74LVC1G125; DESCRIPTION IC Single Buffer With 3-state output -> (none); VALUE 74LVC1G125 -> (none)
- U68: value NTSX2102GU8_1.4X1.2 -> NTSX2102GU8; DESCRIPTION IC Dual supply translating transceiver NTSX2102 -> (none); VALUE NTSX2102GU8 -> (none)
- Y2: value SMD_CRY32.768 -> ECS-.327-CDX-1128; DESCRIPTION CLOCK Crystal 1.5~3.6V ASH7K-32.768KHz-Load Capacitance 6PF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 -> (none); VALUE ECS-.327-CDX-1128 -> (none)
