File: CAD/KiCad/librem5_mainboard/14_GNSS_EXT_CON.kicad_sch (KiCad schematic)
At the start: 54 parts, among them CON1 ANT_CON_3, CON13 600-10429-01_L, J10 CAMERA24PIN035-NFC, U19 TPS78001DRV, U20 BGA725L6, U32 MAX-8, U55 74LVC1G125-SC70-5

Commit message: Use KiCad's new PADS importer/converter tool to go directly from PADS ascii to KiCad 10, place this newly converted project in CAD/PADS/librem5_mainboard/librem5_mainboard_kicad_conversion/, keep the previous converted project that's in CAD/KiCad/librem5_mainboard/ and update it to also use KiCad 10
The one in CAD/KiCad/ seems to be a bit better but this newly converted
project is available in case it might have some improvements (e.g. in
cross-probing or some other more accurate details). Either one (or both)
may be used to completely move the project over to KiCad.

Signed-off-by: Eric Kuzmenko <eric.kuzmenko@puri.sm>
Parts:
- ANT3: value APEX2X2 -> ECT818000500; DESCRIPTION CON RF IV 2X2X0.6 Íâ¾¶1.5 ÄÚ¾¶0.45 -> (none); VALUE ECT818000500 -> (none)
- C100, C255: value C0201 -> 103; DESCRIPTION CAP CER 0.01uF 25V 20% X5R 0201 -> (none); VALUE 103 -> (none)
- C2191, C98, C99: value C0201 -> 105; DESCRIPTION CAP CER 1uF 6V3 20% X5R 0201 -> (none); VALUE 105 -> (none)
- C256, C451, C454, C87: value C0201 -> 56PF; DESCRIPTION CAP CER 56pF 50Vdc 5% C0G C0201 -> (none); VALUE 56PF -> (none)
- C452: value C0201 -> 1nF; DESCRIPTION Ceramic CAP 1nF 25 10% X5R 0201 -> (none); VALUE 1nF -> (none)
- C453, C88: value C0201 -> 120P; DESCRIPTION CAP CER 120PF 25V 10% NPO 0201 -> (none); VALUE 120P -> (none)
- C520: value C0201 -> 104; DESCRIPTION CAP CER 0.1uF 6V3 20% X5R 0201 -> (none); VALUE 104 -> (none)
- C53, C85, C86: value C0201 -> NC; DESCRIPTION Z CAP CER 1uF 6V3 20% X5R 0201 -> (none); VALUE NC -> (none)
- C96, C97: value C0402 -> 4.7UF; DESCRIPTION CAP CER 4.7uF 6V3 20% X5R 0402 -> (none); VALUE 4.7UF -> (none)
- CON1: value ANT_CON_3 -> AT0331-R; VALUE AT0331-R -> (none)
- CON13: value 600-10429-01_L -> (none)
- D19: value DIODE_SCHTKY_0 -> RB751G-40; DESCRIPTION Diode schottky SOD723 40V 30mA mark:5 RB751G-40 ³¤µç -> (none); VALUE RB751G-40 -> (none)
- F5, F9: value FILTER_ESD_BUS4 -> IP4252CZ8-4; DESCRIPTION IC ESD Filter 40 ohm 12pF 4CH -> (none); VALUE IP4252CZ8-4 -> (none)
- J10: value CAMERA24PIN035-NFC -> OK-06F024-04; DESCRIPTION SOCKET Board-to-FPC Ä¸×ù 0.4mm 24pin ºÏ¸ß0.8mm -> (none); VALUE OK-06F024-04 -> (none)
- L11: value BEAD-0402 -> 1 / HPZ1005U121-1R1TF; DESCRIPTION Resistor Chip 0402 1 Ohm 1/16W 1% RALEC -> (none); VALUE 1 / HPZ1005U121-1R1TF -> (none)
- L12: value BEAD-0402 -> NC; DESCRIPTION Z FB 120ohm@100MHz 100ohm@1GHz DCR0.13ohm 1.1A T:0.5mm -> (none); VALUE NC -> (none)
- L25, L26: value BEAD-0201 -> 10; DESCRIPTION FB 240ohm@100MHz DCR0.41ohm 0.35A T:0.3mm -> (none); VALUE 10 -> (none)
- L3: value BEAD-0201 -> 0; DESCRIPTION Resistor Chip 0201 0R Ohm 1/16W 1% RALEC -> (none); VALUE 0 -> (none)
- L68: value BEAD-0201 -> 5.6nh; DESCRIPTION Ceramic inductor,5.6nH¡À0.2nH,250mA,Q18,0.88¦¸,6000MHz,0201 -> (none); VALUE 5.6nh -> (none)
- R106: value RES_2 -> NC; DESCRIPTION Resistor Chip 0201 0R Ohm 1/16W 1% RALEC -> (none); VALUE NC -> (none)
- R120: value RES_2 -> 100K; DESCRIPTION Resistor Chip 0201 100K Ohm 1/16W 1% RALEC -> (none); VALUE 100K -> (none)
- R136: value RES_2 -> 22nH; DESCRIPTION FIXED IND 27NH 160MA 1.6 OHM SMD -> (none); VALUE 22nH -> (none)
- R144, R256: value RES_2 -> 0; DESCRIPTION Resistor Chip 0201 0R Ohm 1/16W 1% RALEC -> (none); VALUE 0 -> (none)
- R146, R150, R178, R59, R60: value RES_2 -> 1K; DESCRIPTION Resistor Chip 0201 1K Ohm 1/16W 1% RALEC -> (none); VALUE 1K -> (none)
- R148, R164, R212, R7: value RES_2 -> 10K; DESCRIPTION Resistor Chip 0201 10K Ohm 1/16W 1% RALEC -> (none); VALUE 10K -> (none)
- R163: value RES_2 -> 16K; DESCRIPTION Resistor Chip 0201 16K Ohm 1/16W 1% RALEC -> (none); VALUE 16K -> (none)
- R249: value R_0201 -> 10K; DESCRIPTION Resistor Chip 0201 10K Ohm 1/16W 1% -> (none); VALUE 10K -> (none)
- TS3: DESCRIPTION Z -> (none); VALUE SC-M1.4 -> (none)
- TV13: value TEST-POINT -> M3; DESCRIPTION Z -> (none); VALUE M3 -> (none)
- U19: DESCRIPTION IC LDO 1.8V-5.5V 150mA 1.2--5.5V IQ:0.5uA -> (none); VALUE TPS78001DRV -> (none)
- U20: DESCRIPTION Silicon Germanium Low Noise Amplifier BGA725L6 -> (none)
- U32: value MAX-8 -> TESEO-LIV3F; DESCRIPTION IC GPS GLONASS, Galileo,BeiDu ,QZSS -> (none); VALUE TESEO-LIV3F -> (none)
- U55: value 74LVC1G125-SC70-5 -> 74LVC1G125; DESCRIPTION IC Single Buffer With 3-state output -> (none); VALUE 74LVC1G125 -> (none)
- Z1: DESCRIPTION SAW RF FILTER B39163B4327P810 -> (none)
