File: CAD/KiCad/librem5_mainboard/15_WIFI_BT.kicad_sch (KiCad schematic)
At the start: 43 parts, among them CON11 ANT_CON1, CON12 ANT_CON1, J5 KEY_E, Q6 2SK3018, Q9 2SK3018, U185 NTBA104_XQFN12, U25 PCMF1USB3S_5P, U40 AP2281

Commit message: Use KiCad's new PADS importer/converter tool to go directly from PADS ascii to KiCad 10, place this newly converted project in CAD/PADS/librem5_mainboard/librem5_mainboard_kicad_conversion/, keep the previous converted project that's in CAD/KiCad/librem5_mainboard/ and update it to also use KiCad 10
The one in CAD/KiCad/ seems to be a bit better but this newly converted
project is available in case it might have some improvements (e.g. in
cross-probing or some other more accurate details). Either one (or both)
may be used to completely move the project over to KiCad.

Signed-off-by: Eric Kuzmenko <eric.kuzmenko@puri.sm>
Parts:
- ANT2: value APEX2X2 -> ECT818000500; DESCRIPTION CON RF IV 2X2X0.6 Íâ¾¶1.5 ÄÚ¾¶0.45 -> (none); VALUE ECT818000500 -> (none)
- C141, C91: value C0201 -> NC; DESCRIPTION Z CAP CER 1uF 6V3 20% X5R 0201 -> (none); VALUE NC -> (none)
- C231, C253, C258, C277, C308, C327: value C0603 -> 22UF; DESCRIPTION CAP CER 22uF 6V3 20% X5R 0603 -> (none); VALUE 22UF -> (none)
- C272, C273: value C0402 -> 4.7UF; DESCRIPTION CAP CER 4.7uF 6V3 20% X5R 0402 -> (none); VALUE 4.7UF -> (none)
- C274, C275, C291, C292, C394, C395: value C0201 -> 105; DESCRIPTION CAP CER 1uF 6V3 20% X5R 0201 -> (none); VALUE 105 -> (none)
- C307, C328: value C0201 -> 104; DESCRIPTION CAP CER 0.1uF 6V3 20% X5R 0201 -> (none); VALUE 104 -> (none)
- C434, C435: value C0402 -> NC; DESCRIPTION CAP CER 10uF 6V3 20% X5R 0402 -> (none); VALUE NC -> (none)
- CON11, CON12: value ANT_CON1 -> AT10-110001-01; DESCRIPTION RF shrapnel,W=1.4mm,L=2.4mm,Hf=1.0¡À0.1mm,Hw=0.55mm µ¯Æ¬ -> (none); VALUE AT10-110001-01 -> (none)
- F10, F11, F6, F8: value FILTER_ESD_BUS4 -> IP4252CZ8-4; DESCRIPTION IC ESD Filter 40 ohm 12pF 4CH -> (none); VALUE IP4252CZ8-4 -> (none)
- J5: value KEY_E -> APCI0136-P001A; DESCRIPTION CON M.2 67PIN E-KEY 0.5mm; H4.8 -> (none); VALUE APCI0136-P001A -> (none)
- L10, L37: value BEAD-0402 -> 0.2 / HPZ1005U121-1R1TF; DESCRIPTION Resistor Chip 0402 0.2 Ohm 1/16W 1% RALEC -> (none); VALUE 0.2 / HPZ1005U121-1R1TF -> (none)
- L35: value BEAD-0201 -> 0; DESCRIPTION Resistor Chip 0201 0R Ohm 1/16W 1% RALEC -> (none); VALUE 0 -> (none)
- Q6, Q9: value 2SK3018 -> RYU002N05; DESCRIPTION TRAN NMOS SW 0.9V DRIVE 50V UMT3 -> (none); VALUE RYU002N05 -> (none)
- R102, R227, R237, R96: value RES_2 -> 47K; DESCRIPTION Resistor Chip 0201 47K Ohm 1/16W 1% RALEC -> (none); VALUE 47K -> (none)
- R97: value RES_2 -> 2.2K; DESCRIPTION Resistor Chip 0201 2.2K Ohm 1/16W 1% RALEC -> (none); VALUE 2.2K -> (none)
- TS5: DESCRIPTION Z -> (none); VALUE SC-M1.4 -> (none)
- TV32: value TEST-POINT -> M3; DESCRIPTION Z -> (none); VALUE M3 -> (none)
- U185: value NTBA104_XQFN12 -> NTB0104GU12; DESCRIPTION IC Dual Supply Buffer 4BIT -> (none); VALUE NTB0104GU12 -> (none)
- U25: value PCMF1USB3S_5P -> PCMF1USB3S; DESCRIPTION IC EMI FILTER FOR DIFF CH W/ ESD PROTECTION 5V WLCSP5 -> (none); VALUE PCMF1USB3S -> (none)
- U40: value AP2281 -> AP2281-3FMG; DESCRIPTION IC SWITCH 80mohm 1.5-6V -> (none); VALUE AP2281-3FMG -> (none)
Changed lines of the file:
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@@
 (kicad_sch
-	(version 20250114)
+	(version 20260306)
 	(generator "eeschema")
-	(generator_version "9.0")
+	(generator_version "10.0")
 	(paper "A2")
 	(title_block
