File: CAD/KiCad/librem5_mainboard/16_4G.kicad_sch (KiCad schematic)
At the start: 69 parts, among them CON7 ANT_CON1, CON8 ANT_CON1, J3 KEY_B, Q1 2SK3018, U12 AP2281, U48 AP2281, U5 NTBA104_XQFN12, U50 TPS22929D, U51 TPS22929D, U9 PCMF1USB3S_5P

Commit message: Use KiCad's new PADS importer/converter tool to go directly from PADS ascii to KiCad 10, place this newly converted project in CAD/PADS/librem5_mainboard/librem5_mainboard_kicad_conversion/, keep the previous converted project that's in CAD/KiCad/librem5_mainboard/ and update it to also use KiCad 10
The one in CAD/KiCad/ seems to be a bit better but this newly converted
project is available in case it might have some improvements (e.g. in
cross-probing or some other more accurate details). Either one (or both)
may be used to completely move the project over to KiCad.

Signed-off-by: Eric Kuzmenko <eric.kuzmenko@puri.sm>
Parts:
- ANT1: value APEX2X2 -> ECT818000500; DESCRIPTION CON RF IV 2X2X0.6 Íâ¾¶1.5 ÄÚ¾¶0.45 -> (none); VALUE ECT818000500 -> (none)
- C220, C245, C246, C247, C248, C281, C283, C290, C299, C306, C329, C330, C335, C336: value C0603 -> 22UF; DESCRIPTION CAP CER 22uF 6V3 20% X5R 0603 -> (none); VALUE 22UF -> (none)
- C225, C226, C257, C298, C346, C347, C348, C350, C436, C437, C439, C440, C441, C442, C443, C444, C94: value C0201 -> 105; DESCRIPTION CAP CER 1uF 6V3 20% X5R 0201 -> (none); VALUE 105 -> (none)
- C270, C271: value C0603 -> NC; DESCRIPTION Z CAP CER 22uF 6V3 20% X5R 0603 -> (none); VALUE NC -> (none)
- C297: value C0402 -> 4.7UF; DESCRIPTION CAP CER 4.7uF 6V3 20% X5R 0402 -> (none); VALUE 4.7UF -> (none)
- C349, C93, C95: value C0201 -> 104; DESCRIPTION CAP CER 0.1uF 6V3 20% X5R 0201 -> (none); VALUE 104 -> (none)
- C89, C90: value C0201 -> NC; DESCRIPTION Z CAP CER 1uF 6V3 20% X5R 0201 -> (none); VALUE NC -> (none)
- CON7, CON8: value ANT_CON1 -> AT10-110001-01; DESCRIPTION RF shrapnel,W=1.4mm,L=2.4mm,Hf=1.0¡À0.1mm,Hw=0.55mm µ¯Æ¬ -> (none); VALUE AT10-110001-01 -> (none)
- F14: value FILTER_ESD_BUS4 -> IP4252CZ8-4; DESCRIPTION IC ESD Filter 40 ohm 12pF 4CH -> (none); VALUE IP4252CZ8-4 -> (none)
- J3: value KEY_B -> APCI0103-P001A; DESCRIPTION CON M.2 67PIN B-KEY 0.5mm; H4.8 -> (none); VALUE APCI0103-P001A -> (none)
- L34: value BEAD-0201 -> 0; DESCRIPTION Resistor Chip 0201 0R Ohm 1/16W 1% RALEC -> (none); VALUE 0 -> (none)
- L36: value BEAD-4030 -> PZ3216D600-4R0TF; DESCRIPTION FB 60ohm@100MHz DCR20mohm 4A T:0.85mm -> (none); VALUE PZ3216D600-4R0TF -> (none)
- Q1: value 2SK3018 -> RYU002N05; DESCRIPTION TRAN NMOS SW 0.9V DRIVE 50V UMT3 -> (none); VALUE RYU002N05 -> (none)
- R101, R158, R159, R160, R83, R84: value RES_2 -> 47K; DESCRIPTION Resistor Chip 0201 47K Ohm 1/16W 1% RALEC -> (none); VALUE 47K -> (none)
- R137: value CURRENT_R -> 20m OHM; DESCRIPTION Resistor Chip 0603 20m Ohm 1/10W 1% RALEC -> (none); VALUE 20m OHM -> (none)
- R228: value RES_2 -> 15K; DESCRIPTION Resistor Chip 0201 15K Ohm 1/16W 1% RALEC -> (none); VALUE 15K -> (none)
- R26: value RES_2 -> 100; DESCRIPTION Resistor Chip 0201 100R Ohm 1/16W 1% RALEC -> (none); VALUE 100 -> (none)
- R261: value R_0201 -> 0R; VALUE 0R -> (none)
- R95: value RES_2 -> 2.2K; DESCRIPTION Resistor Chip 0201 2.2K Ohm 1/16W 1% RALEC -> (none); VALUE 2.2K -> (none)
- TS4: DESCRIPTION Z -> (none); VALUE SC-M1.4 -> (none)
- TV12: value TEST-POINT -> M3; DESCRIPTION Z -> (none); VALUE M3 -> (none)
- TVS21, TVS22, TVS27: value TVS_0402_882 -> PESD3V3S1UL; DESCRIPTION IC ESD 3V3 200pF 30KV SOD882 µ¥Ïò -> (none); VALUE PESD3V3S1UL -> (none)
- U12, U48: value AP2281 -> AP2281-1FMG; DESCRIPTION IC SWITCH 80mohm 1.5-6V -> (none); VALUE AP2281-1FMG -> (none)
- U5: value NTBA104_XQFN12 -> NTB0104GU12; DESCRIPTION IC Dual Supply Buffer 4BIT -> (none); VALUE NTB0104GU12 -> (none)
- U50, U51: value TPS22929D -> NC; DESCRIPTION Z IC SWITCH 80mohm 1.5-6V Controlled Turn-on TPS22929D -> (none); VALUE NC -> (none)
- U9: value PCMF1USB3S_5P -> PCMF1USB3S; DESCRIPTION IC EMI FILTER FOR DIFF CH W/ ESD PROTECTION 5V WLCSP5 -> (none); VALUE PCMF1USB3S -> (none)
Other:
- note removed: "20201204 changed"
