File: CAD/KiCad/librem5_mainboard/17_CAMERA.kicad_sch (KiCad schematic)
At the start: 86 parts, among them J22 CON-34, J4 OK-06F024-04, U11 74LVC1G125-SC70-5, U117 PCMF3USB3S, U134 PCMF3USB3S, U135 PCMF2USB3S_10P, U136 PCMF2USB3S_10P, U21 MIC5233_ADJ_SOT23_5P, U22 74LVC1G125-SC70-5, U33 MIC5233_ADJ_SOT23_5P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

Commit message: Use KiCad's new PADS importer/converter tool to go directly from PADS ascii to KiCad 10, place this newly converted project in CAD/PADS/librem5_mainboard/librem5_mainboard_kicad_conversion/, keep the previous converted project that's in CAD/KiCad/librem5_mainboard/ and update it to also use KiCad 10
The one in CAD/KiCad/ seems to be a bit better but this newly converted
project is available in case it might have some improvements (e.g. in
cross-probing or some other more accurate details). Either one (or both)
may be used to completely move the project over to KiCad.

Signed-off-by: Eric Kuzmenko <eric.kuzmenko@puri.sm>
Parts:
- C200, C228, C230, C301, C302, C323: value C0201 -> 105; DESCRIPTION CAP CER 1uF 6V3 20% X5R 0201 -> (none); VALUE 105 -> (none)
- C227, C229, C250, C251, C252, C276, C70: value C0402 -> 4.7UF; DESCRIPTION CAP CER 4.7uF 6V3 20% X5R 0402 -> (none); VALUE 4.7UF -> (none)
- C300, C43, C449, C526, C54, C65, C7: value C0603 -> 22UF; DESCRIPTION CAP CER 22uF 6V3 20% X5R 0603 -> (none); VALUE 22UF -> (none)
- C345, C534, C63, C64, C84: value C0201 -> 104; DESCRIPTION CAP CER 0.1uF 6V3 20% X5R 0201 -> (none); VALUE 104 -> (none)
- F115, F7: value FILTER_ESD_BUS4 -> IP4252CZ8-4; DESCRIPTION IC ESD Filter 40 ohm 12pF 4CH -> (none); VALUE IP4252CZ8-4 -> (none)
- J22: value CON-34 -> OK-06F034-04; VALUE OK-06F034-04 -> (none)
- J4: DESCRIPTION SOCKET Board-to-FPC Ä¸×ù 0.4mm 24pin ºÏ¸ß0.8mm -> (none); VALUE OK-06F024-04 -> (none)
- L18, L47, L48, L49, L54, L55, L65: value BEAD-0402 -> HPZ1005U121-1R1TF; DESCRIPTION FB 120ohm@100MHz 100ohm@1GHz DCR0.13ohm 1.1A T:0.5mm -> (none); VALUE HPZ1005U121-1R1TF -> (none)
- L27: value BEAD-0402 -> 0.2 / HPZ1005U121-1R1TF; DESCRIPTION Z FB 120ohm@100MHz 100ohm@1GHz DCR0.13ohm 1.1A T:0.5mm -> (none); VALUE 0.2 / HPZ1005U121-1R1TF -> (none)
- L28: value INDUCTOR -> WPN252012H1R0MT; DESCRIPTION IND PWR 1uH@1MHZ 4.2A 20% SMT -> (none); VALUE WPN252012H1R0MT -> (none)
- L44: value BEAD-0402 -> NC; DESCRIPTION Resistor Chip 0402 0.2 Ohm 1/16W 1% RALEC -> (none); VALUE NC -> (none)
- L45: value BEAD-0402 -> 0.2 / HPZ1005U121-1R1TF; DESCRIPTION Resistor Chip 0402 0.2 Ohm 1/16W 1% RALEC -> (none); VALUE 0.2 / HPZ1005U121-1R1TF -> (none)
- L80: value BEAD-0402 -> 1 / HPZ1005U121-1R1TF; DESCRIPTION Resistor Chip 0402 1 Ohm 1/16W 1% RALEC -> (none); VALUE 1 / HPZ1005U121-1R1TF -> (none)
- R11, R12, R32, R69, R8, R9: value RES_2 -> 10K; DESCRIPTION Resistor Chip 0201 10K Ohm 1/16W 1% RALEC -> (none); VALUE 10K -> (none)
- R121, R128: value RES_2 -> 1K; DESCRIPTION Resistor Chip 0201 1K Ohm 1/16W 1% RALEC -> (none); VALUE 1K -> (none)
- R122: value RES_2 -> 27K; DESCRIPTION Resistor Chip 0201 27K Ohm 1/16W 1% RALEC -> (none); VALUE 27K -> (none)
- R123, R131: value RES_2 -> 47K; DESCRIPTION Resistor Chip 0201 47K Ohm 1/16W 1% RALEC -> (none); VALUE 47K -> (none)
- R138: value CURRENT_R -> 20m OHM; DESCRIPTION Resistor Chip 0603 20m Ohm 1/10W 1% RALEC -> (none); VALUE 20m OHM -> (none)
- R234: value RES_2 -> 0R; DESCRIPTION Resistor Chip 0201 499 Ohm 1/16W 1% RALEC -> (none); VALUE 0R -> (none)
- R253: value RES_2 -> NC; DESCRIPTION Resistor Chip 0201 10K Ohm 1/16W 1% RALEC -> (none); VALUE NC -> (none)
- R254: value RES_2 -> 0; DESCRIPTION Resistor Chip 0201 0 Ohm 1/20W 1% RALEC -> (none); VALUE 0 -> (none)
- R33: value RES_2 -> 11.8K; DESCRIPTION Resistor Chip 0201 5.23K Ohm 1/16W 1% RALEC -> (none); VALUE 11.8K -> (none)
- R70: value RES_2 -> 9.09K; DESCRIPTION Resistor Chip 0201 2.2K Ohm 1/16W 1% RALEC -> (none); VALUE 9.09K -> (none)
- R88: value RES_2 -> 12K; DESCRIPTION Resistor Chip 0201 12K Ohm 1/16W 1% RALEC -> (none); VALUE 12K -> (none)
- R89: value RES_2 -> 30.1K; DESCRIPTION Resistor Chip 0201 30.1K Ohm 1/16W 1% RALEC -> (none); VALUE 30.1K -> (none)
- TP92, TP93, TP94, TV17, TV19, TV33, TV53, TV6: value TEST-POINT -> M3; DESCRIPTION Z -> (none); VALUE M3 -> (none)
- TVS53, TVS54, TVS55, TVS56, TVS6, TVS7: value TVS_0402_882 -> PESD3V3S1UL; DESCRIPTION IC ESD 3V3 200pF 30KV SOD882 µ¥Ïò -> (none); VALUE PESD3V3S1UL -> (none)
- U11, U22: value 74LVC1G125-SC70-5 -> 74LVC1G125; DESCRIPTION IC Single Buffer With 3-state output -> (none); VALUE 74LVC1G125 -> (none)
- U117, U134: DESCRIPTION IC EMI FILTER FOR DIFF CH W/ ESD PROTECTION 5V WLCSP15 -> (none); VALUE PCMF3USB3S -> (none)
- U135, U136: value PCMF2USB3S_10P -> PCMF2USB3S; DESCRIPTION IC EMI FILTER FOR DIFF CH W/ ESD PROTECTION 5V WLCSP10 -> (none); VALUE PCMF2USB3S -> (none)
- U21, U37: value MIC5233_ADJ_SOT23_5P -> TLV75801PDBVR; DESCRIPTION IC LDO 1.8V-5.5V 150mA 0.8--5.5V -> (none); VALUE TLV75801PDBVR -> (none)
- U33: value MIC5233_ADJ_SOT23_5P -> LDCL015MR; DESCRIPTION IC LDO 1.8V-5.5V 150mA 0.8--5.5V -> (none); VALUE LDCL015MR -> (none)
- U38: value AP2281 -> AP2281-1FMG; DESCRIPTION IC SWITCH 80mohm 1.5-6V -> (none); VALUE AP2281-1FMG -> (none)
- U7: value ME6211C__M5G -> ME6211C28M5G; DESCRIPTION IC Voltage LDO sot23-5 0.5A Vin:5.5V Vout:2.8V MARK:G1 or S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 -> (none); VALUE ME6211C28M5G -> (none)
- U8: DESCRIPTION IC FLASH Driver Dual 1A -> (none); VALUE LM3560 -> (none)
