File: CAD/KiCad/librem5_mainboard/18_TFT_TP_MOTO.kicad_sch (KiCad schematic)
At the start: 72 parts, among them J6 OK-06F034-04, U17 TPS65132, U29 PCMF3USB3S, U41 AP2281, U42 LM36922-1, U45 PCMF2USB3S_10P

Commit message: Use KiCad's new PADS importer/converter tool to go directly from PADS ascii to KiCad 10, place this newly converted project in CAD/PADS/librem5_mainboard/librem5_mainboard_kicad_conversion/, keep the previous converted project that's in CAD/KiCad/librem5_mainboard/ and update it to also use KiCad 10
The one in CAD/KiCad/ seems to be a bit better but this newly converted
project is available in case it might have some improvements (e.g. in
cross-probing or some other more accurate details). Either one (or both)
may be used to completely move the project over to KiCad.

Signed-off-by: Eric Kuzmenko <eric.kuzmenko@puri.sm>
Parts:
- C239, C249, C341, C60, C61, C62, C69: value C0402 -> 225; DESCRIPTION CAP CER 2.2uF 35V 20% X5R 0402 -> (none); VALUE 225 -> (none)
- C269, C286, C303, C73, C74: value C0402 -> 4.7UF; DESCRIPTION CAP CER 4.7uF 6V3 20% X5R 0402 -> (none); VALUE 4.7UF -> (none)
- C304, C75: value C0201 -> 105; DESCRIPTION CAP CER 1uF 6V3 20% X5R 0201 -> (none); VALUE 105 -> (none)
- C305: value C0603 -> 224; DESCRIPTION CAP CER 0.22uF 35V 20% X5R 0603 -> (none); VALUE 224 -> (none)
- C340, C342, C545: value C0201 -> 103; DESCRIPTION CAP CER 0.01uF 25V 20% X5R 0201 -> (none); VALUE 103 -> (none)
- C344: value C0201 -> 104; DESCRIPTION CAP CER 0.1uF 6V3 20% X5R 0201 -> (none); VALUE 104 -> (none)
- C76: value C0603 -> 225; DESCRIPTION CAP CER 2.2uF 35V 20% X5R 0603 -> (none); VALUE 225 -> (none)
- D10: value PTVS24VS1UR -> PTVS30VS1UR; DESCRIPTION IC TVS 30V 400W -> (none); VALUE PTVS30VS1UR -> (none)
- D2: value ZLLS400 -> B5817WS; DESCRIPTION DIODE Schottky Barrier Diode SOD323 -> (none); VALUE B5817WS -> (none)
- F4: value FILTER_ESD_BUS4 -> IP4252CZ8-4; DESCRIPTION IC ESD Filter 40 ohm 12pF 4CH -> (none); VALUE IP4252CZ8-4 -> (none)
- J6: DESCRIPTION SOCKET Board-to-FPC Ä¸×ù 0.4mm 34pin ºÏ¸ß0.8mm -> (none); VALUE OK-06F034-04 -> (none)
- L20: value INDUCTOR -> WPN252012H100MT; DESCRIPTION IND PWR10uH@1MHZ 1.35A 20% SMT -> (none); VALUE WPN252012H100MT -> (none)
- L21: value INDUCTOR -> WPN252012H3R3MT; DESCRIPTION IND PWR 3.3uH@1MHZ 1.9A 20% SMT -> (none); VALUE WPN252012H3R3MT -> (none)
- L31, L40, L41, L42: value BEAD-0402 -> HPZ1005U121-1R1TF; DESCRIPTION FB 120ohm@100MHz 100ohm@1GHz DCR0.13ohm 1.1A T:0.5mm -> (none); VALUE HPZ1005U121-1R1TF -> (none)
- L43, L52: value BEAD-0201 -> PZ0603D241-R35TF; DESCRIPTION FB 240ohm@100MHz DCR0.41ohm 0.35A T:0.3mm -> (none); VALUE PZ0603D241-R35TF -> (none)
- L76, L77: value BEAD-0402 -> 0.2 / HPZ1005U121-1R1TF; DESCRIPTION Resistor Chip 0402 0.2 Ohm 1/16W 1% RALEC -> (none); VALUE 0.2 / HPZ1005U121-1R1TF -> (none)
- L8: value BEAD-0402 -> 1 / HPZ1005U121-1R1TF; DESCRIPTION Resistor Chip 0402 1 Ohm 1/16W 1% RALEC -> (none); VALUE 1 / HPZ1005U121-1R1TF -> (none)
- R107, R17, R23, R235, R24, R53: value RES_2 -> 10K; DESCRIPTION Resistor Chip 0201 10K Ohm 1/16W 1% RALEC -> (none); VALUE 10K -> (none)
- R119, R142, R51, R85, R86: value RES_2 -> 1K; DESCRIPTION Resistor Chip 0201 1K Ohm 1/16W 1% RALEC -> (none); VALUE 1K -> (none)
- R124, R49, R50, R87: value RES_2 -> 0; DESCRIPTION Resistor Chip 0201 0R Ohm 1/16W 1% RALEC -> (none); VALUE 0 -> (none)
- R133: value RES_2 -> 47K; DESCRIPTION Resistor Chip 0201 47K Ohm 1/16W 1% RALEC -> (none); VALUE 47K -> (none)
- R71, R72: value RES_2 -> 100K; DESCRIPTION Resistor Chip 0201 100K Ohm 1/16W 1% RALEC -> (none); VALUE 100K -> (none)
- TC10, TC3, TC7, TC9, TV15, TV16, TV52: value TEST-POINT -> M3; DESCRIPTION Z -> (none); VALUE M3 -> (none)
- TVS1, TVS2, TVS24, TVS25, TVS26: value TVS_0402_882 -> PESD3V3S1UL; DESCRIPTION IC ESD 3V3 200pF 30KV SOD882 µ¥Ïò -> (none); VALUE PESD3V3S1UL -> (none)
- TVS23, TVS28: value TVS_0402_882 -> PESD12VV1BL; DESCRIPTION IC ESD 5V0 45pF 30KV SOD882 Ë«Ïò -> (none); VALUE PESD12VV1BL -> (none)
- U17: value TPS65132 -> TPS65132B5; DESCRIPTION IC VREG +-5.5V Dual Output -> (none); VALUE TPS65132B5 -> (none)
- U29: DESCRIPTION IC EMI FILTER FOR DIFF CH W/ ESD PROTECTION 5V WLCSP15 -> (none); VALUE PCMF3USB3S -> (none)
- U41: value AP2281 -> AP2281-3FMG; DESCRIPTION IC SWITCH 80mohm 1.5-6V -> (none); VALUE AP2281-3FMG -> (none)
- U42: value LM36922-1 -> LM36922; DESCRIPTION IC High-Brightness,Dual-string White LED Driver -> (none); VALUE LM36922 -> (none)
- U45: value PCMF2USB3S_10P -> PCMF2USB3S; DESCRIPTION IC EMI FILTER FOR DIFF CH W/ ESD PROTECTION 5V WLCSP10 -> (none); VALUE PCMF2USB3S -> (none)
