File: CAD/KiCad/librem5_mainboard/19_USB_HUB_SD.kicad_sch (KiCad schematic)
At the start: 42 parts, among them J7 SIM-CARD-SA2101110135-01, Q13 2SK3018, Q3 2SK3018, U2 USB2642, U43 AP2281, U44 AP2281, Y3 XTAL_13Y

Commit message: Use KiCad's new PADS importer/converter tool to go directly from PADS ascii to KiCad 10, place this newly converted project in CAD/PADS/librem5_mainboard/librem5_mainboard_kicad_conversion/, keep the previous converted project that's in CAD/KiCad/librem5_mainboard/ and update it to also use KiCad 10
The one in CAD/KiCad/ seems to be a bit better but this newly converted
project is available in case it might have some improvements (e.g. in
cross-probing or some other more accurate details). Either one (or both)
may be used to completely move the project over to KiCad.

Signed-off-by: Eric Kuzmenko <eric.kuzmenko@puri.sm>
Parts:
- C142, C293, C309, C314, C338, C353, C355, C66, C71, C72: value C0201 -> 104; DESCRIPTION CAP CER 0.1uF 6V3 20% X5R 0201 -> (none); VALUE 104 -> (none)
- C222, C337, C382: value C0402 -> 4.7UF; DESCRIPTION CAP CER 4.7uF 6V3 20% X5R 0402 -> (none); VALUE 4.7UF -> (none)
- C386, C390: value C0201 -> 105; DESCRIPTION CAP CER 1uF 6V3 20% X5R 0201 -> (none); VALUE 105 -> (none)
- C391, C392: value C0201 -> 18PF; DESCRIPTION CAP CER 18PF 25V 20% NPO 0201 -> (none); VALUE 18PF -> (none)
- C67: value C0603 -> 22UF; DESCRIPTION CAP CER 22uF 6V3 20% X5R 0603 -> (none); VALUE 22UF -> (none)
- F1, F13, F3: value FILTER_ESD_BUS4 -> IP4252CZ8-4; DESCRIPTION IC ESD Filter 40 ohm 12pF 4CH -> (none); VALUE IP4252CZ8-4 -> (none)
- L79: value BEAD-0402 -> 0.2 / HPZ1005U121-1R1TF; DESCRIPTION Resistor Chip 0402 0.2 Ohm 1/16W 1% RALEC -> (none); VALUE 0.2 / HPZ1005U121-1R1TF -> (none)
- Q13, Q3: value 2SK3018 -> RYU002N05; DESCRIPTION TRAN NMOS SW 0.9V DRIVE 50V UMT3 -> (none); VALUE RYU002N05 -> (none)
- R198: value RES_2 -> NC; DESCRIPTION Z Resistor Chip 0201 10K Ohm 1/16W 1% RALEC -> (none); VALUE NC -> (none)
- R218, R37, R46, R55: value RES_2 -> 47K; DESCRIPTION Resistor Chip 0201 47K Ohm 1/16W 1% RALEC -> (none); VALUE 47K -> (none)
- R263: value R_0201 -> 10K; VALUE 10K -> (none)
- R38: value CURRENT_R -> 20m OHM; DESCRIPTION Resistor Chip 0603 20m Ohm 1/10W 1% RALEC -> (none); VALUE 20m OHM -> (none)
- R40: value RES_2 -> 12K; DESCRIPTION Resistor Chip 0201 12K Ohm 1/16W 1% RALEC -> (none); VALUE 12K -> (none)
- R41: value RES_2 -> 0R; DESCRIPTION Resistor Chip 0201 47K Ohm 1/16W 1% RALEC -> (none); VALUE 0R -> (none)
- R42: value RES_2 -> 1M; DESCRIPTION Resistor Chip 0201 1M Ohm 1/16W 1% RALEC -> (none); VALUE 1M -> (none)
- TV31: value TEST-POINT -> M3; DESCRIPTION Z -> (none); VALUE M3 -> (none)
- TVS10, TVS4: value TVS_0402_882 -> PESD3V3S1UL; DESCRIPTION IC ESD 3V3 200pF 30KV SOD882 µ¥Ïò -> (none); VALUE PESD3V3S1UL -> (none)
- U2: value USB2642 -> usb2642; DESCRIPTION IC USB 2.0 High Speed 2-Port Hub with SD Reader Controller -> (none); VALUE usb2642 -> (none)
- U43, U44: value AP2281 -> AP2281-3FMG; DESCRIPTION IC SWITCH 80mohm 1.5-6V -> (none); VALUE AP2281-3FMG -> (none)
- Y3: value XTAL_13Y -> 24MHz; DESCRIPTION CLOCK Crystal 24MHz 18pF +-20PPM/ -> (none); VALUE 24MHz -> (none)
