File: CAD/KiCad/librem5_mainboard/20_AUDIO_WM8962.kicad_sch (KiCad schematic)
At the start: 102 parts, among them J2 JACK-JA-36A1-111, Q12 2SK3018, Q2 2SK3018, U24 WM8962, U31 3SM222FMT1KA, U46 AP2281, U510 NC7WZ17, U78 MIC5233_ADJ_SOT23_5P

Commit message: Use KiCad's new PADS importer/converter tool to go directly from PADS ascii to KiCad 10, place this newly converted project in CAD/PADS/librem5_mainboard/librem5_mainboard_kicad_conversion/, keep the previous converted project that's in CAD/KiCad/librem5_mainboard/ and update it to also use KiCad 10
The one in CAD/KiCad/ seems to be a bit better but this newly converted
project is available in case it might have some improvements (e.g. in
cross-probing or some other more accurate details). Either one (or both)
may be used to completely move the project over to KiCad.

Signed-off-by: Eric Kuzmenko <eric.kuzmenko@puri.sm>
Parts:
- C1251, C260, C294, C30, C310, C37, C39, C45, C47, C59, C852: value C0402 -> 4.7UF; DESCRIPTION CAP CER 4.7uF 6V3 20% X5R 0402 -> (none); VALUE 4.7UF -> (none)
- C1323, C295, C296, C326, C38, C40, C42, C58, C901: value C0201 -> 105; DESCRIPTION CAP CER 1uF 6V3 20% X5R 0201 -> (none); VALUE 105 -> (none)
- C25, C26, C325, C44: value C0201 -> 104; DESCRIPTION CAP CER 0.1uF 6V3 20% X5R 0201 -> (none); VALUE 104 -> (none)
- C259: value C0201 -> NC; DESCRIPTION Z CAP CER 1uF 6V3 20% X5R 0201 -> (none); VALUE NC -> (none)
- C324: value C0603 -> 22UF; DESCRIPTION CAP CER 22uF 6V3 20% X5R 0603 -> (none); VALUE 22UF -> (none)
- C41: value C0603 -> NC; DESCRIPTION Z CAP CER 22uF 6V3 20% X5R 0603 -> (none); VALUE NC -> (none)
- J2: value JACK-JA-36A1-111 -> JA-36A2-111; VALUE JA-36A2-111 -> (none)
- L1, L14: value BEAD-0402 -> HPZ1005U121-1R1TF; DESCRIPTION FB 120ohm@100MHz 100ohm@1GHz DCR0.13ohm 1.1A T:0.5mm -> (none); VALUE HPZ1005U121-1R1TF -> (none)
- L16: value BEAD-0402 -> 1 / HPZ1005U121-1R1TF; DESCRIPTION Resistor Chip 0402 1 Ohm 1/16W 1% RALEC -> (none); VALUE 1 / HPZ1005U121-1R1TF -> (none)
- L17: value BEAD-0402 -> 10 / HPZ1005U121-1R1TF; DESCRIPTION Resistor Chip 0402 10 Ohm 1/16W 1% RALEC -> (none); VALUE 10 / HPZ1005U121-1R1TF -> (none)
- L2: value BEAD-0402 -> NC; DESCRIPTION Z FB 120ohm@100MHz 100ohm@1GHz DCR0.13ohm 1.1A T:0.5mm -> (none); VALUE NC -> (none)
- L4, L5, L53, L6, L66, L67, L92: value BEAD0603 -> MZAH1608G471-1R6TF; DESCRIPTION FB 470ohm@100MHz 350ohm@1GHz DCR0.075ohm 1.6A T:0.8mm -> (none); VALUE MZAH1608G471-1R6TF -> (none)
- L50, L51, L61: value BEAD-0402 -> MZAH1005F352-R27TF; DESCRIPTION FB 3500ohm@100MHz 1600ohm@1GHz DCR1ohm 270mA T:0.5mm -> (none); VALUE MZAH1005F352-R27TF -> (none)
- L7: value BEAD-0402 -> 0.2 / HPZ1005U121-1R1TF; DESCRIPTION Resistor Chip 0402 0.2 Ohm 1/16W 1% RALEC -> (none); VALUE 0.2 / HPZ1005U121-1R1TF -> (none)
- Q12: value 2SK3018 -> BSS138PW; DESCRIPTION TRAN NMOS SW 0.9V DRIVE 50V UMT3 -> (none); VALUE BSS138PW -> (none)
- Q2: value 2SK3018 -> RYU002N05; DESCRIPTION TRAN NMOS SW 0.9V DRIVE 50V UMT3 -> (none); VALUE RYU002N05 -> (none)
- R10, R13, R14, R16, R18, R43, R44, R525, R552: value RES_2 -> 33; DESCRIPTION Resistor Chip 0201 33R Ohm 1/16W 1% RALEC -> (none); VALUE 33 -> (none)
- R109, R166: value RES_2 -> 0R; DESCRIPTION Resistor Chip 0201 1K Ohm 1/16W 1% RALEC -> (none); VALUE 0R -> (none)
- R125: value RES_2 -> 47K; DESCRIPTION Resistor Chip 0201 47K Ohm 1/16W 1% RALEC -> (none); VALUE 47K -> (none)
- R129: value RES_2 -> 2.2K; DESCRIPTION Resistor Chip 0201 2.2K Ohm 1/16W 1% RALEC -> (none); VALUE 2.2K -> (none)
- R149: value RES_2 -> 10K; DESCRIPTION Resistor Chip 0201 10K Ohm 1/16W 1% RALEC -> (none); VALUE 10K -> (none)
- R187, R2101, R47, R569, R573, R65: value RES_2 -> 0; DESCRIPTION Resistor Chip 0201 0R Ohm 1/16W 1% RALEC -> (none); VALUE 0 -> (none)
- R188, R25, R564, R565: value RES_2 -> NC; DESCRIPTION Z Resistor Chip 0201 10K Ohm 1/16W 1% RALEC -> (none); VALUE NC -> (none)
- R250: value R_0201 -> 47K; DESCRIPTION Resistor Chip 0201 10K Ohm 1/16W 1% RALEC -> (none); VALUE 47K -> (none)
- R258: value RES_2 -> NC; DESCRIPTION Resistor Chip 0201 33R Ohm 1/16W 1% RALEC -> (none); VALUE NC -> (none)
- R288: value RES_2 -> 15K; DESCRIPTION Resistor Chip 0201 15K Ohm 1/16W 1% RALEC -> (none); VALUE 15K -> (none)
- R289: value RES_2 -> 30.1K; DESCRIPTION Resistor Chip 0201 30.1K Ohm 1/16W 1% RALEC -> (none); VALUE 30.1K -> (none)
- R39: value SDR -> (none); DESCRIPTION Z -> (none)
- R5: value RES_2 -> 10R; DESCRIPTION Resistor Chip 0201 1K Ohm 1/16W 1% RALEC -> (none); VALUE 10R -> (none)
- R529, R545: value RES_2 -> 100K; DESCRIPTION Resistor Chip 0201 100K Ohm 1/16W 1% RALEC -> (none); VALUE 100K -> (none)
- R554: value RES_2 -> 47K; DESCRIPTION Resistor Chip 0201 10K Ohm 1/16W 1% RALEC -> (none); VALUE 47K -> (none)
- R58: value RES_2 -> 27K; DESCRIPTION Resistor Chip 0201 27K Ohm 1/16W 1% RALEC -> (none); VALUE 27K -> (none)
- TP22, TP23: value T_POINT_R -> U1_DN; DESCRIPTION Z -> (none); VALUE U1_DN -> (none)
- TP25, TP26, TP27, TP48, TV18, TV50, TV51: value TEST-POINT -> M3; DESCRIPTION Z -> (none); VALUE M3 -> (none)
- TVS17, TVS18, TVS5, TVS9: value TVS_0402_882 -> PESD3V3S1UL; DESCRIPTION IC ESD 3V3 200pF 30KV SOD882 µ¥Ïò -> (none); VALUE PESD3V3S1UL -> (none)
- TVS3, TVS52, TVS58, TVS59: value TVS_0402_882 -> PESD5V0S1BL; DESCRIPTION IC ESD 5V0 45pF 30KV SOD882 Ë«Ïò -> (none); VALUE PESD5V0S1BL -> (none)
- U24: DESCRIPTION IC AUDIO Stereo CODEC -> (none); VALUE WM8962 -> (none)
- U31: DESCRIPTION IC CMOS MEMS microphone -> (none); VALUE 3SM222FMT1KA -> (none)
- U46: value AP2281 -> AP2281-3FMG; DESCRIPTION IC SWITCH 80mohm 1.5-6V -> (none); VALUE AP2281-3FMG -> (none)
- U510: value NC7WZ17 -> NC; DESCRIPTION Z IC Dual Buffer with Schmit MicroPak NC7WZ17L6X -> (none); VALUE NC -> (none)
- U78: value MIC5233_ADJ_SOT23_5P -> LDCL015MR; DESCRIPTION IC LDO 1.8V-5.5V 150mA 0.8--5.5V -> (none); VALUE LDCL015MR -> (none)
