File: CAD/KiCad/librem5_mainboard/21_DEBUG_MFG.kicad_sch (KiCad schematic)
At the start: 90 parts

Commit message: Use KiCad's new PADS importer/converter tool to go directly from PADS ascii to KiCad 10, place this newly converted project in CAD/PADS/librem5_mainboard/librem5_mainboard_kicad_conversion/, keep the previous converted project that's in CAD/KiCad/librem5_mainboard/ and update it to also use KiCad 10
The one in CAD/KiCad/ seems to be a bit better but this newly converted
project is available in case it might have some improvements (e.g. in
cross-probing or some other more accurate details). Either one (or both)
may be used to completely move the project over to KiCad.

Signed-off-by: Eric Kuzmenko <eric.kuzmenko@puri.sm>
Parts:
- D7: value DIODE_SCHTKY_0 -> RB751G-40; DESCRIPTION Diode schottky SOD723 40V 30mA mark:5 RB751G-40 ³¤µç -> (none); VALUE RB751G-40 -> (none)
- E1, E10, E11, E12, E13, E14, E15, E16, E17, E18, E19, E2, E20, E21, E22, E23, E24, E25, E26, E27, E28, E29, E3, E30, E31, E32, E33, E34, E35, E36, E37, E4, E5, E6, E7, E8, E9: value PTC3121N -> (none)
- JV1, JV2: value CLIP-1.1H -> (none)
- R169, R170: value RES_2 -> 10K; DESCRIPTION Resistor Chip 0201 10K Ohm 1/16W 1% RALEC -> (none); VALUE 10K -> (none)
- R171, R172, R173, R246: value RES_2 -> NC; DESCRIPTION Z Resistor Chip 0201 10K Ohm 1/16W 1% RALEC -> (none); VALUE NC -> (none)
- R174, R175: value RES_2 -> 1K; DESCRIPTION Resistor Chip 0201 1K Ohm 1/16W 1% RALEC -> (none); VALUE 1K -> (none)
- R176: value RES_2 -> 100; DESCRIPTION Resistor Chip 0201 100R Ohm 1/16W 1% RALEC -> (none); VALUE 100 -> (none)
- R247: value RES_2 -> 0; DESCRIPTION Resistor Chip 0201 0R Ohm 1/16W 1% RALEC -> (none); VALUE 0 -> (none)
- TP10, TP33, TP4, TP40: value T_POINT_R -> GND; DESCRIPTION Z -> (none); VALUE GND -> (none)
- TP11: value T_POINT_R -> BAT; DESCRIPTION Z -> (none); VALUE BAT -> (none)
- TP12: value T_POINT_R -> U1_DN; DESCRIPTION Z -> (none); VALUE U1_DN -> (none)
- TP16, TP17: value TP-60MIL -> (none)
- TP2: value T_POINT_R -> SMC_IO; DESCRIPTION Z -> (none); VALUE SMC_IO -> (none)
- TP28: value T_POINT_R -> U1_DP; DESCRIPTION Z -> (none); VALUE U1_DP -> (none)
- TP29: value T_POINT_R -> M4_UR2; DESCRIPTION Z -> (none); VALUE M4_UR2 -> (none)
- TP3: value T_POINT_R -> SMC_CK; DESCRIPTION Z -> (none); VALUE SMC_CK -> (none)
- TP30: value T_POINT_R -> M4_UT2; DESCRIPTION Z -> (none); VALUE M4_UT2 -> (none)
- TP31, TP32, TP36: value T_POINT_R -> 8M_UT1; DESCRIPTION Z -> (none); VALUE 8M_UT1 -> (none)
- TP34: value T_POINT_R -> VBUS1; DESCRIPTION Z -> (none); VALUE VBUS1 -> (none)
- TP35: value T_POINT_R -> 8M_UR1; DESCRIPTION Z -> (none); VALUE 8M_UR1 -> (none)
- TP37: value T_POINT_R -> BM0; DESCRIPTION Z -> (none); VALUE BM0 -> (none)
- TP38: value T_POINT_R -> BM1; DESCRIPTION Z -> (none); VALUE BM1 -> (none)
- TP39: value T_POINT_R -> 3V3; DESCRIPTION Z -> (none); VALUE 3V3 -> (none)
- TP41: value T_POINT_R -> TCK; DESCRIPTION Z -> (none); VALUE TCK -> (none)
- TP42: value T_POINT_R -> TMS; DESCRIPTION Z -> (none); VALUE TMS -> (none)
- TP43: value T_POINT_R -> TDI; DESCRIPTION Z -> (none); VALUE TDI -> (none)
- TP44: value T_POINT_R -> TDO; DESCRIPTION Z -> (none); VALUE TDO -> (none)
- TP45: value T_POINT_R -> J_RST; DESCRIPTION Z -> (none); VALUE J_RST -> (none)
- TP46: value T_POINT_R -> J_PORB; DESCRIPTION Z -> (none); VALUE J_PORB -> (none)
- TP47: value T_POINT_R -> NTC; DESCRIPTION Z -> (none); VALUE NTC -> (none)
- TP5: value T_POINT_R -> SMC_P; DESCRIPTION Z -> (none); VALUE SMC_P -> (none)
- TP501: value T_POINT_R -> U1_ID; DESCRIPTION Z -> (none); VALUE U1_ID -> (none)
- TP6: value T_POINT_R -> SMC_BOOT0; DESCRIPTION Z -> (none); VALUE SMC_BOOT0 -> (none)
- TS1, TS2: value SC-M2 -> NC; DESCRIPTION Z SCREEN M.2¹Ì¶¨ÂÝÄ¸ M3 Ö±¾¶5.5MM H:3MM ×Ü¸ß:3.7MM -> (none); VALUE NC -> (none)
- TS15, TS16, TS17, TS6, TS7, TS8, TS9: DESCRIPTION Z -> (none); VALUE SC-M1.4 -> (none)
