File: CAD/KiCad/librem5_mainboard/librem5_mainboard.kicad_sch (KiCad schematic)
At the start: 0 parts

Commit message: KiCad Mainboard: Rename all sheets to correctly follow the sheet numbering
Update the project to KiCad 8.99

Signed-off-by: Eric Kuzmenko <eric.kuzmenko@puri.sm>
Other:
- sheet C-03_POWER_TREE renamed 02_POWER_TREE
- sheet C-04_CPU_PWR renamed 03_CPU_PWR
- sheet C-05_LPDDR4 renamed 04_LPDDR4
- sheet C-06_CPU_IO renamed 05_CPU_IO
- sheet C-07_CPU_MISC_RTC renamed 06_CPU_MISC_RTC
- sheet C-08_CPU_PHY renamed 07_CPU_PHY
- sheet C-09_EMMC renamed 08_EMMC
- sheet C-10_PMIC renamed 09_PMIC
- sheet C-11_BOOT_CFG renamed 10_BOOT_CFG
- sheet C-12_USB_TYPE-C renamed 11_USB_TYPE-C
- sheet C-13_CHARGE_BAT_LED renamed 12_CHARGE_BAT_LED
- sheet C-14_SENSOR_SMARTCARD renamed 13_SENSOR_SMARTCARD
- sheet C-15_GNSS_EXT_CON renamed 14_GNSS_EXT_CON
- sheet C-16_WIFI_BT renamed 15_WIFI_BT
- sheet C-17_4G renamed 16_4G
- sheet C-18_CAMERA renamed 17_CAMERA
- sheet C-19_TFT_TP_MOTO renamed 18_TFT_TP_MOTO
- sheet C-20_USB_HUB_SD renamed 19_USB_HUB_SD
- sheet C-21_AUDIO_WM8962 renamed 20_AUDIO_WM8962
- sheet C-22_DEBUG_MFG renamed 21_DEBUG_MFG
- sheet 02_POWER_TREE: file C-03_POWER_TREE.kicad_sch -> 02_POWER_TREE.kicad_sch
- sheet 03_CPU_PWR: file C-04_CPU_PWR.kicad_sch -> 03_CPU_PWR.kicad_sch
- sheet 04_LPDDR4: file C-05_LPDDR4.kicad_sch -> 04_LPDDR4.kicad_sch
- sheet 05_CPU_IO: file C-06_CPU_IO.kicad_sch -> 05_CPU_IO.kicad_sch
- sheet 06_CPU_MISC_RTC: file C-07_CPU_MISC_RTC.kicad_sch -> 06_CPU_MISC_RTC.kicad_sch
- sheet 07_CPU_PHY: file C-08_CPU_PHY.kicad_sch -> 07_CPU_PHY.kicad_sch
- sheet 08_EMMC: file C-09_EMMC.kicad_sch -> 08_EMMC.kicad_sch
- sheet 09_PMIC: file C-10_PMIC.kicad_sch -> 09_PMIC.kicad_sch
- sheet 10_BOOT_CFG: file C-11_BOOT_CFG.kicad_sch -> 10_BOOT_CFG.kicad_sch
- sheet 11_USB_TYPE-C: file C-12_USB_TYPE-C.kicad_sch -> 11_USB_TYPE-C.kicad_sch
- sheet 12_CHARGE_BAT_LED: file C-13_CHARGE_BAT_LED.kicad_sch -> 12_CHARGE_BAT_LED.kicad_sch
- sheet 13_SENSOR_SMARTCARD: file C-14_SENSOR_SMARTCARD.kicad_sch -> 13_SENSOR_SMARTCARD.kicad_sch
- sheet 14_GNSS_EXT_CON: file C-15_GNSS_EXT_CON.kicad_sch -> 14_GNSS_EXT_CON.kicad_sch
- sheet 15_WIFI_BT: file C-16_WIFI_BT.kicad_sch -> 15_WIFI_BT.kicad_sch
- sheet 16_4G: file C-17_4G.kicad_sch -> 16_4G.kicad_sch
- sheet 17_CAMERA: file C-18_CAMERA.kicad_sch -> 17_CAMERA.kicad_sch
- sheet 18_TFT_TP_MOTO: file C-19_TFT_TP_MOTO.kicad_sch -> 18_TFT_TP_MOTO.kicad_sch
- sheet 19_USB_HUB_SD: file C-20_USB_HUB_SD.kicad_sch -> 19_USB_HUB_SD.kicad_sch
- sheet 20_AUDIO_WM8962: file C-21_AUDIO_WM8962.kicad_sch -> 20_AUDIO_WM8962.kicad_sch
- sheet 21_DEBUG_MFG: file C-22_DEBUG_MFG.kicad_sch -> 21_DEBUG_MFG.kicad_sch
Changed lines of the file:
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@@
 (kicad_sch
-	(version 20231120)
+	(version 20241004)
 	(generator "eeschema")
-	(generator_version "8.0")
+	(generator_version "8.99")
 	(paper "A1")
 	(title_block
@@
 		(at 563.88 508)
 		(size 12.7 3.81)
+		(exclude_from_sim no)
+		(in_bom yes)
+		(on_board yes)
+		(dnp no)
 		(fields_autoplaced yes)
 		(stroke
@@
 			(color 0 0 0 0.0000)
 		)
-		(property "Sheetname" "C-17_4G"
+		(property "Sheetname" "16_4G"
 			(at 563.88 507.2884 0)
 			(effects
@@
 			)
 		)
-		(property "Sheetfile" "C-17_4G.kicad_sch"
+		(property "Sheetfile" "16_4G.kicad_sch"
 			(at 563.88 512.3946 0)
 			(effects
@@
 		(at 495.3 508)
 		(size 12.7 3.81)
+		(exclude_from_sim no)
+		(in_bom yes)
+		(on_board yes)
+		(dnp no)
 		(fields_autoplaced yes)
 		(stroke
@@
 			(color 0 0 0 0.0000)
 		)
-		(property "Sheetname" "C-15_GNSS_EXT_CON"
+		(property "Sheetname" "14_GNSS_EXT_CON"
 			(at 495.3 507.2884 0)
 			(effects
@@
 			)
 		)
-		(property "Sheetfile" "C-15_GNSS_EXT_CON.kicad_sch"
+		(property "Sheetfile" "14_GNSS_EXT_CON.kicad_sch"
 			(at 495.3 512.3946 0)
 			(effects
@@
 		(at 287.02 508)
 		(size 12.7 3.81)
+		(exclude_from_sim no)
+		(in_bom yes)
+		(on_board yes)
+		(dnp no)
 		(fields_autoplaced yes)
 		(stroke
@@
 			(color 0 0 0 0.0000)
 		)
-		(property "Sheetname" "C-09_EMMC"
+		(property "Sheetname" "08_EMMC"
 			(at 287.02 507.2884 0)
 			(effects
@@
 			)
 		)
-		(property "Sheetfile" "C-09_EMMC.kicad_sch"
+		(property "Sheetfile" "08_EMMC.kicad_sch"
 			(at 287.02 512.3946 0)
 			(effects
@@
 		(at 255.27 508)
 		(size 12.7 3.81)
+		(exclude_from_sim no)
+		(in_bom yes)
+		(on_board yes)
+		(dnp no)
 		(fields_autoplaced yes)
 		(stroke
@@
 			(color 0 0 0 0.0000)
 		)
-		(property "Sheetname" "C-08_CPU_PHY"
+		(property "Sheetname" "07_CPU_PHY"
 			(at 255.27 507.2884 0)
 			(effects
@@
 			)
 		)
-		(property "Sheetfile" "C-08_CPU_PHY.kicad_sch"
+		(property "Sheetfile" "07_CPU_PHY.kicad_sch"
 			(at 255.27 512.3946 0)
 			(effects
@@
 		(at 157.48 508)
 		(size 12.7 3.81)
+		(exclude_from_sim no)
+		(in_bom yes)
+		(on_board yes)
+		(dnp no)
 		(fields_autoplaced yes)
 		(stroke
@@
 			(color 0 0 0 0.0000)
 		)
-		(property "Sheetname" "C-05_LPDDR4"
+		(property "Sheetname" "04_LPDDR4"
 			(at 157.48 507.2884 0)
 			(effects
@@
 			)
 		)
-		(property "Sheetfile" "C-05_LPDDR4.kicad_sch"
+		(property "Sheetfile" "04_LPDDR4.kicad_sch"
 			(at 157.48 512.3946 0)
 			(effects
@@
 		(at 589.28 508)
 		(size 12.7 3.81)
+		(exclude_from_sim no)
+		(in_bom yes)
+		(on_board yes)
+		(dnp no)
 		(fields_autoplaced yes)
 		(stroke
@@
 			(color 0 0 0 0.0000)
 		)
-		(property "Sheetname" "C-18_CAMERA"
+		(property "Sheetname" "17_CAMERA"
 			(at 589.28 507.2884 0)
 			(effects
@@
 			)
 		)
-		(property "Sheetfile" "C-18_CAMERA.kicad_sch"
+		(property "Sheetfile" "17_CAMERA.kicad_sch"
 			(at 589.28 512.3946 0)
 			(effects
@@
 		(at 728.98 508)
 		(size 12.7 3.81)
+		(exclude_from_sim no)
+		(in_bom yes)
+		(on_board yes)
+		(dnp no)
 		(fields_autoplaced yes)
 		(stroke
@@
 			(color 0 0 0 0.0000)
 		)
-		(property "Sheetname" "C-22_DEBUG_MFG"
+		(property "Sheetname" "21_DEBUG_MFG"
 			(at 728.98 507.2884 0)
 			(effects
@@
 			)
 		)
-		(property "Sheetfile" "C-22_DEBUG_MFG.kicad_sch"
+		(property "Sheetfile" "21_DEBUG_MFG.kicad_sch"
 			(at 728.98 512.3946 0)
 			(effects
@@
 		(at 452.12 508)
 		(size 12.7 3.81)
+		(exclude_from_sim no)
+		(in_bom yes)
+		(on_board yes)
+		(dnp no)
 		(fields_autoplaced yes)
 		(stroke
@@
 			(color 0 0 0 0.0000)
 		)
-		(property "Sheetname" "C-14_SENSOR_SMARTCARD"
+		(property "Sheetname" "13_SENSOR_SMARTCARD"
 			(at 452.12 507.2884 0)
 			(effects
@@
 			)
 		)
-		(property "Sheetfile" "C-14_SENSOR_SMARTCARD.kicad_sch"
+		(property "Sheetfile" "13_SENSOR_SMARTCARD.kicad_sch"
 			(at 452.12 512.3946 0)
 			(effects
@@
 		(at 690.88 508)
 		(size 12.7 3.81)
+		(exclude_from_sim no)
+		(in_bom yes)
+		(on_board yes)
+		(dnp no)
 		(fields_autoplaced yes)
 		(stroke
@@
 			(color 0 0 0 0.0000)
 		)
-		(property "Sheetname" "C-21_AUDIO_WM8962"
+		(property "Sheetname" "20_AUDIO_WM8962"
 			(at 690.88 507.2884 0)
 			(effects
@@
 			)
 		)
-		(property "Sheetfile" "C-21_AUDIO_WM8962.kicad_sch"
+		(property "Sheetfile" "20_AUDIO_WM8962.kicad_sch"
 			(at 690.88 512.3946 0)
 			(effects
@@
 		(at 344.17 508)
 		(size 12.7 3.81)
+		(exclude_from_sim no)
+		(in_bom yes)
+		(on_board yes)
+		(dnp no)
 		(fields_autoplaced yes)
 		(stroke
@@
 			(color 0 0 0 0.0000)
 		)
-		(property "Sheetname" "C-11_BOOT_CFG"
+		(property "Sheetname" "10_BOOT_CFG"
 			(at 344.17 507.2884 0)
 			(effects
@@
 			)
 		)
-		(property "Sheetfile" "C-11_BOOT_CFG.kicad_sch"
+		(property "Sheetfile" "10_BOOT_CFG.kicad_sch"
 			(at 344.17 512.3946 0)
 			(effects
@@
 		(at 412.75 508)
 		(size 12.7 3.81)
+		(exclude_from_sim no)
+		(in_bom yes)
+		(on_board yes)
+		(dnp no)
 		(fields_autoplaced yes)
 		(stroke
@@
 			(color 0 0 0 0.0000)
 		)
-		(property "Sheetname" "C-13_CHARGE_BAT_LED"
+		(property "Sheetname" "12_CHARGE_BAT_LED"
 			(at 412.75 507.2884 0)
 			(effects
@@
 			)
 		)
-		(property "Sheetfile" "C-13_CHARGE_BAT_LED.kicad_sch"
+		(property "Sheetfile" "12_CHARGE_BAT_LED.kicad_sch"
 			(at 412.75 512.3946 0)
 			(effects
@@
 		(at 218.44 508)
 		(size 12.7 3.81)
+		(exclude_from_sim no)
+		(in_bom yes)
+		(on_board yes)
+		(dnp no)
 		(fields_autoplaced yes)
 		(stroke
@@
 			(color 0 0 0 0.0000)
 		)
-		(property "Sheetname" "C-07_CPU_MISC_RTC"
+		(property "Sheetname" "06_CPU_MISC_RTC"
 			(at 218.44 507.2884 0)
 			(effects
@@
 			)
 		)
-		(property "Sheetfile" "C-07_CPU_MISC_RTC.kicad_sch"
+		(property "Sheetfile" "06_CPU_MISC_RTC.kicad_sch"
 			(at 218.44 512.3946 0)
 			(effects
@@
 		(at 655.32 508)
 		(size 12.7 3.81)
+		(exclude_from_sim no)
+		(in_bom yes)
+		(on_board yes)
+		(dnp no)
 		(fields_autoplaced yes)
 		(stroke
@@
 			(color 0 0 0 0.0000)
 		)
-		(property "Sheetname" "C-20_USB_HUB_SD"
+		(property "Sheetname" "19_USB_HUB_SD"
 			(at 655.32 507.2884 0)
 			(effects
@@
 			)
 		)
-		(property "Sheetfile" "C-20_USB_HUB_SD.kicad_sch"
+		(property "Sheetfile" "19_USB_HUB_SD.kicad_sch"
 			(at 655.32 512.3946 0)
 			(effects
@@
 		(at 90.17 508)
 		(size 12.7 3.81)
+		(exclude_from_sim no)
+		(in_bom yes)
+		(on_board yes)
+		(dnp no)
 		(fields_autoplaced yes)
 		(stroke
@@
 			(color 0 0 0 0.0000)
 		)
-		(property "Sheetname" "C-03_POWER_TREE"
+		(property "Sheetname" "02_POWER_TREE"
 			(at 90.17 507.2884 0)
 			(effects
@@
 			)
 		)
-		(property "Sheetfile" "C-03_POWER_TREE.kicad_sch"
+		(property "Sheetfile" "02_POWER_TREE.kicad_sch"
 			(at 90.17 512.3946 0)
 			(effects
@@
 		(at 316.23 508)
 		(size 12.7 3.81)
+		(exclude_from_sim no)
+		(in_bom yes)
+		(on_board yes)
+		(dnp no)
 		(fields_autoplaced yes)
 		(stroke
@@
 			(color 0 0 0 0.0000)
 		)
-		(property "Sheetname" "C-10_PMIC"
+		(property "Sheetname" "09_PMIC"
 			(at 316.23 507.2884 0)
 			(effects
@@
 			)
 		)
-		(property "Sheetfile" "C-10_PMIC.kicad_sch"
+		(property "Sheetfile" "09_PMIC.kicad_sch"
 			(at 316.23 512.3946 0)
 			(effects
@@
 		(at 533.4 508)
 		(size 12.7 3.81)
+		(exclude_from_sim no)
+		(in_bom yes)
+		(on_board yes)
+		(dnp no)
 		(fields_autoplaced yes)
 		(stroke
@@
 			(color 0 0 0 0.0000)
 		)
-		(property "Sheetname" "C-16_WIFI_BT"
+		(property "Sheetname" "15_WIFI_BT"
 			(at 533.4 507.2884 0)
 			(effects
@@
 			)
 		)
-		(property "Sheetfile" "C-16_WIFI_BT.kicad_sch"
+		(property "Sheetfile" "15_WIFI_BT.kicad_sch"
 			(at 533.4 512.3946 0)
 			(effects
@@
 		(at 619.76 508)
 		(size 12.7 3.81)
+		(exclude_from_sim no)
+		(in_bom yes)
+		(on_board yes)
+		(dnp no)
 		(fields_autoplaced yes)
 		(stroke
@@
 			(color 0 0 0 0.0000)
 		)
-		(property "Sheetname" "C-19_TFT_TP_MOTO"
+		(property "Sheetname" "18_TFT_TP_MOTO"
 			(at 619.76 507.2884 0)
 			(effects
@@
 			)
 		)
-		(property "Sheetfile" "C-19_TFT_TP_MOTO.kicad_sch"
+		(property "Sheetfile" "18_TFT_TP_MOTO.kicad_sch"
 			(at 619.76 512.3946 0)
 			(effects
@@
 		(at 377.19 508)
 		(size 12.7 3.81)
+		(exclude_from_sim no)
+		(in_bom yes)
+		(on_board yes)
+		(dnp no)
 		(fields_autoplaced yes)
 		(stroke
@@
 			(color 0 0 0 0.0000)
 		)
-		(property "Sheetname" "C-12_USB_TYPE-C"
+		(property "Sheetname" "11_USB_TYPE-C"
 			(at 377.19 507.2884 0)
 			(effects
@@
 			)
 		)
-		(property "Sheetfile" "C-12_USB_TYPE-C.kicad_sch"
+		(property "Sheetfile" "11_USB_TYPE-C.kicad_sch"
 			(at 377.19 512.3946 0)
 			(effects
@@
 		(at 125.73 508)
 		(size 12.7 3.81)
+		(exclude_from_sim no)
+		(in_bom yes)
+		(on_board yes)
+		(dnp no)
 		(fields_autoplaced yes)
 		(stroke
@@
 			(color 0 0 0 0.0000)
 		)
-		(property "Sheetname" "C-04_CPU_PWR"
+		(property "Sheetname" "03_CPU_PWR"
 			(at 125.73 507.2884 0)
 			(effects
@@
 			)
 		)
-		(property "Sheetfile" "C-04_CPU_PWR.kicad_sch"
+		(property "Sheetfile" "03_CPU_PWR.kicad_sch"
 			(at 125.73 512.3946 0)
 			(effects
@@
 		(at 187.96 508)
 		(size 12.7 3.81)
+		(exclude_from_sim no)
+		(in_bom yes)
+		(on_board yes)
+		(dnp no)
 		(fields_autoplaced yes)
 		(stroke
@@
 			(color 0 0 0 0.0000)
 		)
-		(property "Sheetname" "C-06_CPU_IO"
+		(property "Sheetname" "05_CPU_IO"
 			(at 187.96 507.2884 0)
 			(effects
@@
 			)
 		)
-		(property "Sheetfile" "C-06_CPU_IO.kicad_sch"
+		(property "Sheetfile" "05_CPU_IO.kicad_sch"
 			(at 187.96 512.3946 0)
 			(effects
@@
 		)
 	)
+	(embedded_fonts no)
 )
